File: modules/05_VCO/VCO.kicad_pcb (KiCad board)
At the start: 2 copper layers, 160 x 200 mm, 5 parts, among them J1 BUS CONNECTOR

Commit message: panel updates & vco
Parts:
- removed H1, H2, H3, H4: MountingHole, FormantKO:MountingHole_2.7mm_M2.5
- added C1: 1n, FormantKO:C_Disc, F.Cu at (110.1, 56.4)
- added C10: 100µ, FormantKO:CP_Axial_600, F.Cu at (85.4, 264.4)
- added C11: 100µ, FormantKO:CP_Axial_600, F.Cu at (85.4, 270.8)
- added C12: 680n, FormantKO:C_Disc, F.Cu at (80.7, 276.0)
- added C13: 1n, FormantKO:C_Disc, F.Cu at (115.2, 147.9)
- added C2: 3n3, FormantKO:C_Disc, F.Cu at (120.2, 74.2)
- added C3: 680n, FormantKO:C_Disc, F.Cu at (163.4, 193.0)
- added C4: 680n, FormantKO:C_Disc, F.Cu at (163.4, 197.1)
- added C5: 680n, FormantKO:C_Disc, F.Cu at (163.4, 201.2)
- added C6: 680n, FormantKO:C_Disc, F.Cu at (51.7, 142.8)
- added C7: 680n, FormantKO:C_Disc, F.Cu at (148.2, 188.5)
- added C8: 680n, FormantKO:C_Disc, F.Cu at (132.9, 150.4)
- added C9: 47µ, FormantKO:CP_Axial_600, F.Cu at (122.8, 104.7)
- added D1: DUS, FormantKO:DUS, F.Cu at (158.3, 56.4)
- added D2: DUS, FormantKO:DUS, F.Cu at (158.3, 69.1)
- added D3: DUG, FormantKO:DUG, F.Cu at (112.6, 114.8)
- added D4: DUG, FormantKO:DUG, F.Cu at (132.9, 114.8)
- added D5: DUS, FormantKO:DUS, F.Cu at (115.2, 196.1)
- added D6: DUS, FormantKO:DUS, F.Cu at (115.2, 188.5)
- added D7: DUS, FormantKO:DUS, F.Cu at (163.4, 135.2)
- added D8: Panel_LED, FormantKO:Panel_Connector_1x02, F.Cu at (33.9, 159.3)
- added IC1: 7413, FormantKO:DIP-14, F.Cu at (145.6, 47.5)
- added IC10: µA741C, FormantKO:DIP-8, F.Cu at (73.2, 194.8)
- added IC11: µA741C, FormantKO:DIP-8, F.Cu at (116.4, 210.1)
- added IC2: µA741C, FormantKO:DIP-8, F.Cu at (119.0, 57.7)
- added IC3: µA726, Package_TO_SOT_THT:TO-5-10, F.Cu at (95.4, 56.2)
- added IC4: µA741C, FormantKO:DIP-8, F.Cu at (70.7, 52.6)
- added IC5: µA741C, FormantKO:DIP-8, F.Cu at (149.4, 133.9)
- added IC6: µA741C, FormantKO:DIP-8, F.Cu at (124.0, 172.0)
- added IC7: µA741C, FormantKO:DIP-8, F.Cu at (149.4, 172.0)
- added IC8: µA741C, FormantKO:DIP-8, F.Cu at (66.9, 130.1)
- added IC9: µA741C, FormantKO:DIP-8, F.Cu at (61.8, 165.6)
- added J2: KOV SELECT, FormantKO:Jumper_1x03, F.Cu at (171.0, 133.5)
- added J3: IOS SELECT, Connector_PinHeader_2.54mm:PinHeader_2x03_P2.54mm_Vertical, F.Cu at (166.0, 206.3)
- added J5: Mono_Jack, FormantKO:Panel_Connector_1x02, F.Cu at (42.8, 79.6)
- added J6: Mono_Jack, FormantKO:Panel_Connector_1x02, F.Cu at (33.9, 85.7)
- added J7: Mono_Jack, FormantKO:Panel_Connector_1x02, F.Cu at (73.5, 249.0)
- added J8: Mono_Jack, FormantKO:Panel_Connector_1x02, F.Cu at (73.5, 256.8)
- added MH1: CardBracket, FormantKO:Card_Bracket, F.Cu at (25.0, 175.0)
- added MH2: CardBracket, FormantKO:Card_Bracket, F.Cu at (25.0, 75.0)
- added P1: 100k, FormantKO:Panel_Connector_1x03, F.Cu at (33.9, 41.2)
- added P10: 4k7, FormantKO:Potentiometer_Trimmer, F.Cu at (168.5, 74.2)
- added P11: 100k, FormantKO:Potentiometer_Trimmer, F.Cu at (163.4, 117.4)
- added P12: 10k, FormantKO:Potentiometer_Trimmer, F.Cu at (122.8, 122.4)
- added P13: 100k, FormantKO:Potentiometer_Trimmer, F.Cu at (135.5, 201.2)
- added P14: 100k, FormantKO:Potentiometer_Trimmer, F.Cu at (83.7, 243.3)
- added P15: 100k, FormantKO:Potentiometer_Trimmer, F.Cu at (83.7, 254.4)
- added P2: 100k, FormantKO:Panel_Connector_1x03, F.Cu at (33.9, 53.8)
- added P3: 50k, FormantKO:Panel_Connector_1x03, F.Cu at (33.0, 70.7)
- added P4: 100k, FormantKO:Panel_Connector_1x03, F.Cu at (33.9, 109.7)
- added P5: 10k, FormantKO:Panel_Connector_1x03, F.Cu at (33.9, 142.8)
- added P6: 4k7, FormantKO:Panel_Connector_1x03, F.Cu at (62.8, 256.8)
- added P7: 200R, FormantKO:Potentiometer_Trimmer, F.Cu at (111.3, 37.5)
- added P8: 100k, FormantKO:Potentiometer_Trimmer, F.Cu at (82.2, 66.6)
- added P9: 2k2, FormantKO:Potentiometer_Trimmer, F.Cu at (112.6, 76.7)
- added R1: 150k, FormantKO:R_Axial_Horizontal, F.Cu at (52.9, 43.7)
- added R10: 100k, FormantKO:R_Axial_Horizontal, F.Cu at (68.2, 64.0)
- added R11: 1M, FormantKO:R_Axial_Horizontal, F.Cu at (108.8, 48.8)
- added R12: 68k, FormantKO:R_Axial_Horizontal, F.Cu at (103.7, 43.7)
- added R13: 200k, FormantKO:R_Axial_Horizontal, F.Cu at (96.1, 66.6)
- added R14: 1M, FormantKO:R_Axial_Horizontal, F.Cu at (127.9, 50.1)
- added R15: 330R, FormantKO:R_Axial_Horizontal, F.Cu at (139.3, 74.2)
- added R16: 4k7, FormantKO:R_Axial_Horizontal, F.Cu at (83.4, 84.4)
- added R17: 12k, FormantKO:R_Axial_Horizontal, F.Cu at (97.4, 78.0)
- added R18: 1k78, FormantKO:R_Axial_Horizontal, F.Cu at (153.3, 70.4)
- added R19: 1k, FormantKO:R_Axial_Horizontal, F.Cu at (141.8, 59.0)
- added R2: 100k, FormantKO:R_Axial_Horizontal, F.Cu at (55.5, 48.8)
- added R20: 12k, FormantKO:R_Axial_Horizontal, F.Cu at (58.0, 74.2)
- added R21: 33k, FormantKO:R_Axial_Horizontal, F.Cu at (153.3, 116.1)
- added R22: 22k, FormantKO:R_Axial_Horizontal, F.Cu at (148.2, 116.1)
- added R23: 120k, FormantKO:R_Axial_Horizontal, F.Cu at (158.3, 133.9)
- added R24: 47k, FormantKO:R_Axial_Horizontal, F.Cu at (158.3, 172.0)
- added R25: 12k, FormantKO:R_Axial_Horizontal, F.Cu at (150.7, 151.7)
- added R26: 120k, FormantKO:R_Axial_Horizontal, F.Cu at (55.5, 206.3)
- added R27: 180k, FormantKO:R_Axial_Horizontal, F.Cu at (55.5, 201.2)
- added R28: 5k6, FormantKO:R_Axial_Horizontal, F.Cu at (106.3, 137.7)
- added R29: 5k6, FormantKO:R_Axial_Horizontal, F.Cu at (106.3, 152.9)
- added R3: 150k, FormantKO:R_Axial_Horizontal, F.Cu at (41.5, 50.1)
- added R30: 4k7, FormantKO:R_Axial_Horizontal, F.Cu at (130.4, 131.3)
- added R31: 1k, FormantKO:R_Axial_Horizontal, F.Cu at (136.8, 145.3)
- added R32: 47R, FormantKO:R_Axial_Horizontal, F.Cu at (113.9, 142.8)
- added R33: 47R, FormantKO:R_Axial_Horizontal, F.Cu at (113.9, 163.1)
- added R34: 47R, FormantKO:R_Axial_Horizontal, F.Cu at (113.9, 158.0)
- added R35: 1k, FormantKO:R_Axial_Horizontal, F.Cu at (136.8, 155.5)
- added R36: 10k, FormantKO:R_Axial_Horizontal, F.Cu at (135.5, 131.3)
- added R37: 330k, FormantKO:R_Axial_Horizontal, F.Cu at (136.8, 160.6)
- added R38: 1k, FormantKO:R_Axial_Horizontal, F.Cu at (129.1, 188.5)
- added R39: 22k, FormantKO:R_Axial_Horizontal, F.Cu at (116.4, 183.4)
- added R4: 100R, FormantKO:R_Axial_Horizontal, F.Cu at (44.0, 62.8)
- added R40: 1k, FormantKO:R_Axial_Horizontal, F.Cu at (116.4, 201.2)
- added R41: 3k9, FormantKO:R_Axial_Horizontal, F.Cu at (125.3, 210.1)
- added R42: 150k, FormantKO:R_Axial_Horizontal, F.Cu at (55.5, 196.1)
- added R43: 150k, FormantKO:R_Axial_Horizontal, F.Cu at (55.5, 191.0)
- added R44: 100k, FormantKO:R_Axial_Horizontal, F.Cu at (48.9, 228.1)
- added R45: 470R, FormantKO:R_Axial_Horizontal, F.Cu at (48.9, 232.2)
- added R46: 3k9, FormantKO:R_Axial_Horizontal, F.Cu at (48.9, 236.2)
- added R47: 10k, FormantKO:R_Axial_Horizontal, F.Cu at (48.9, 240.3)
- added R48: 10k, FormantKO:R_Axial_Horizontal, F.Cu at (48.9, 244.3)
- added R49: 10k, FormantKO:R_Axial_Horizontal, F.Cu at (48.9, 248.4)
- added R5: 47k, FormantKO:R_Axial_Horizontal, F.Cu at (55.5, 53.9)
- added R50: 10k, FormantKO:R_Axial_Horizontal, F.Cu at (48.9, 252.4)
- added R51: 10k, FormantKO:R_Axial_Horizontal, F.Cu at (48.9, 256.5)
- added R52: 10k, FormantKO:R_Axial_Horizontal, F.Cu at (48.9, 260.5)
- added R53: 180R, FormantKO:R_Axial_Horizontal, F.Cu at (48.9, 264.6)
- added R54: 220k, FormantKO:R_Axial_Horizontal, F.Cu at (48.9, 268.6)
- added R55: 22k, FormantKO:R_Axial_Horizontal, F.Cu at (48.9, 272.7)
- added R56: 100k, FormantKO:R_Axial_Horizontal, F.Cu at (48.9, 276.7)
- added R57: 100k, FormantKO:R_Axial_Horizontal, F.Cu at (48.9, 280.8)
- added R58: 68k, FormantKO:R_Axial_Horizontal, F.Cu at (48.9, 284.8)
- added R59: 15k, FormantKO:R_Axial_Horizontal, F.Cu at (48.9, 288.9)
- added R6: 2k37, FormantKO:R_Axial_Horizontal, F.Cu at (70.7, 43.7)
- added R7: 1k5, FormantKO:R_Axial_Horizontal, F.Cu at (68.2, 69.1)
- added R8: 750R, FormantKO:R_Axial_Horizontal, F.Cu at (89.8, 55.1)
- added R9: 100k, FormantKO:R_Axial_Horizontal, F.Cu at (55.5, 59.0)
- added S1: ~, FormantKO:Panel_Connector_1x03, F.Cu at (33.9, 97.1)
- added S2: ~, FormantKO:Panel_Connector_1x03, F.Cu at (62.8, 264.6)
- added S3: ~, FormantKO:Panel_Connector_1x03, F.Cu at (33.9, 208.8)
- added S4: ~, FormantKO:Panel_Connector_1x03, F.Cu at (33.9, 170.7)
- added S5: ~, FormantKO:Panel_Connector_1x03, F.Cu at (33.9, 183.4)
- added S6: ~, FormantKO:Panel_Connector_1x03, F.Cu at (33.9, 196.1)
- added T1: TUN, FormantKO:TO-18, F.Cu at (126.6, 74.2)
- added T2: N-FET, FormantKO:TO-92, F.Cu at (102.5, 76.7)
- added T3: N-FET, FormantKO:TO-92, F.Cu at (72.0, 84.4)
- added T4: TUN, FormantKO:TO-18, F.Cu at (117.7, 133.9)
- added T5: TUN, FormantKO:TO-18, F.Cu at (124.0, 152.9)
- added T6: TUN, FormantKO:TO-18, F.Cu at (72.7, 265.0)
- added T7: TUN, FormantKO:TO-18, F.Cu at (72.7, 272.2)
- added T8: TUP, FormantKO:TO-18, F.Cu at (72.7, 279.5)
- J1: value BUS CONNECTOR -> Card_Connector; footprint FormantKO:DIN_Male -> FormantKO:Card_Connector
- moved J1 69.4 mm to (185.0, 175.0), turned to 0 degrees
Other:
- board text removed: "INCOMPLETE"
