File: panels/DUAL_VCA/DUAL_VCA.kicad_sch (KiCad schematic)
At the start: 4 parts

Commit message: updated adsr/dual vca
Other:
- company: THE HOUSE OF GALAHAD -> (none)
- title: DUAL VCA -> (none)
Changed lines of the file:
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@@
 	(generator "eeschema")
 	(generator_version "10.0")
-	(paper "USLetter")
-	(title_block
-		(title "DUAL VCA")
-		(rev "A")
-		(company "THE HOUSE OF GALAHAD")
-		(comment 1 "FORMANT-KO")
-	)
+	(paper "A4")
 	(symbol
 		(lib_id "FormantKO:Mounting_Hole")
