File: panels/RFM/RFM.kicad_pcb (KiCad board)
At the start: 2 copper layers, 70.8 x 261.8 mm, 19 parts

Commit message: 3U panels
Other:
- board text added: "ƒ_{0}"
- board text removed: "f_{0}"

Commit message: panel templates, rfm
Parts:
- added REF**: Arrow, FormantKO-Panel:Arrow, F.Cu at (212.6, 50.2)
Changed lines of the file:
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@@
 		(capping no)
 		(filling no)
-		(grid_origin 201.635894 150.240428)
+		(grid_origin 166.245894 19.365428)
 		(pcbplotparams
 			(layerselection 0x00000000_00000000_55555555_5755f5ff)
@@
 		)
 	)
+	(footprint "FormantKO-Panel:Arrow"
+		(layer "F.Cu")
+		(at 212.635894 50.240428 90)
+		(property "Reference" "REF**"
+			(at 0 -0.5 90)
+			(unlocked yes)
+			(layer "F.SilkS")
+			(hide yes)
+			(effects
+				(font
+					(size 1 1)
+					(thickness 0.1)
+				)
+			)
+		)
+		(property "Value" "Arrow"
+			(at 0 1 90)
+			(unlocked yes)
+			(layer "F.Fab")
+			(hide yes)
+			(effects
+				(font
+					(size 1 1)
+					(thickness 0.15)
+				)
+			)
+		)
+		(property "Datasheet" ""
+			(at 0 0 90)
+			(unlocked yes)
+			(layer "F.Fab")
+			(hide yes)
+			(effects
+				(font
+					(size 1 1)
+					(thickness 0.15)
+				)
+			)
+		)
+		(property "Description" ""
+			(at 0 0 90)
+			(unlocked yes)
+			(layer "F.Fab")
+			(hide yes)
+			(effects
+				(font
+					(size 1 1)
+					(thickness 0.15)
+				)
+			)
+		)
+		(attr smd)
+		(duplicate_pad_numbers_are_jumpers no)
+		(fp_poly
+			(pts
+				(xy 0 0) (xy -1.5 -2) (xy 1.5 -2)
+			)
+			(stroke
+				(width 0.1)
+				(type solid)
+			)
+			(fill yes)
+			(layer "F.SilkS")
+		)
+		(embedded_fonts no)
+	)
 	(footprint "FormantKO-Panel:CardBracket"
 		(layer "F.Cu")
@@
 		)
 	)
-	(gr_poly
-		(pts
-			(xy 211.635894 50.240428) (xy 208.635894 47.240428) (xy 208.635894 53.240428)
-		)
-		(stroke
-			(width 0.1)
-			(type solid)
-		)
-		(fill yes)
-		(layer "F.SilkS")
-	)
 	(gr_rect
