File: panels/VCF_12/VCF_12.kicad_pcb (KiCad board)
At the start: 2 copper layers, 70.8 x 261.8 mm, 20 parts

Commit message: 3U panels
Other:
- outline, holes or cut-outs redrawn
- board text removed: "BIG TEXT"
- board text removed: "NORMAL TEXT"
- board text removed: "SMALLER TEXT"
- board text removed: "TINY TEXT"

Commit message: panel templates, rfm
Parts:
- added REF**: Arrow, FormantKO-Panel:Arrow, F.Cu at (201.6, 61.2)
- added REF**: Arrow, FormantKO-Panel:Arrow, F.Cu at (218.6, 96.2)
- added REF**: Arrow, FormantKO-Panel:Arrow, F.Cu at (184.6, 96.2)
Changed lines of the file:
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@@
 		)
+	)
+	(footprint "FormantKO-Panel:Arrow"
+		(layer "F.Cu")
+		(at 184.635894 96.240428)
+		(property "Reference" "REF**"
+			(at 0 -0.5 0)
+			(unlocked yes)
+			(layer "F.SilkS")
+			(hide yes)
+			(effects
+				(font
+					(size 1 1)
+					(thickness 0.1)
+				)
+			)
+		)
+		(property "Value" "Arrow"
+			(at 0 1 0)
+			(unlocked yes)
+			(layer "F.Fab")
+			(hide yes)
+			(effects
+				(font
+					(size 1 1)
+					(thickness 0.15)
+				)
+			)
+		)
+		(property "Datasheet" ""
+			(at 0 0 0)
+			(unlocked yes)
+			(layer "F.Fab")
+			(hide yes)
+			(effects
+				(font
+					(size 1 1)
+					(thickness 0.15)
+				)
+			)
+		)
+		(property "Description" ""
+			(at 0 0 0)
+			(unlocked yes)
+			(layer "F.Fab")
+			(hide yes)
+			(effects
+				(font
+					(size 1 1)
+					(thickness 0.15)
+				)
+			)
+		)
+		(attr smd)
+		(duplicate_pad_numbers_are_jumpers no)
+		(fp_poly
+			(pts
+				(xy 0 0) (xy -1.5 -2) (xy 1.5 -2)
+			)
+			(stroke
+				(width 0.1)
+				(type solid)
+			)
+			(fill yes)
+			(layer "F.SilkS")
+		)
+		(embedded_fonts no)
 	)
 	(footprint "FormantKO-Panel:PanelMountingHole"
@@
 		)
 	)
+	(footprint "FormantKO-Panel:Arrow"
+		(layer "F.Cu")
+		(at 201.635894 61.240428)
+		(property "Reference" "REF**"
+			(at 0 -0.5 0)
+			(unlocked yes)
+			(layer "F.SilkS")
+			(hide yes)
+			(effects
+				(font
+					(size 1 1)
+					(thickness 0.1)
+				)
+			)
+		)
+		(property "Value" "Arrow"
+			(at 0 1 0)
+			(unlocked yes)
+			(layer "F.Fab")
+			(hide yes)
+			(effects
+				(font
+					(size 1 1)
+					(thickness 0.15)
+				)
+			)
+		)
+		(property "Datasheet" ""
+			(at 0 0 0)
+			(unlocked yes)
+			(layer "F.Fab")
+			(hide yes)
+			(effects
+				(font
+					(size 1 1)
+					(thickness 0.15)
+				)
+			)
+		)
+		(property "Description" ""
+			(at 0 0 0)
+			(unlocked yes)
+			(layer "F.Fab")
+			(hide yes)
+			(effects
+				(font
+					(size 1 1)
+					(thickness 0.15)
+				)
+			)
+		)
+		(attr smd)
+		(duplicate_pad_numbers_are_jumpers no)
+		(fp_poly
+			(pts
+				(xy 0 0) (xy -1.5 -2) (xy 1.5 -2)
+			)
+			(stroke
+				(width 0.1)
+				(type solid)
+			)
+			(fill yes)
+			(layer "F.SilkS")
+		)
+		(embedded_fonts no)
+	)
 	(footprint "FormantKO-Panel:PanelMountingHole"
 		(layer "F.Cu")
@@
 		)
 	)
+	(footprint "FormantKO-Panel:Arrow"
+		(layer "F.Cu")
+		(at 218.635894 96.240428)
+		(property "Reference" "REF**"
+			(at 0 -0.5 0)
+			(unlocked yes)
+			(layer "F.SilkS")
+			(hide yes)
+			(effects
+				(font
+					(size 1 1)
+					(thickness 0.1)
+				)
+			)
+		)
+		(property "Value" "Arrow"
+			(at 0 1 0)
+			(unlocked yes)
+			(layer "F.Fab")
+			(hide yes)
+			(effects
+				(font
+					(size 1 1)
+					(thickness 0.15)
+				)
+			)
+		)
+		(property "Datasheet" ""
+			(at 0 0 0)
+			(unlocked yes)
+			(layer "F.Fab")
+			(hide yes)
+			(effects
+				(font
+					(size 1 1)
+					(thickness 0.15)
+				)
+			)
+		)
+		(property "Description" ""
+			(at 0 0 0)
+			(unlocked yes)
+			(layer "F.Fab")
+			(hide yes)
+			(effects
+				(font
+					(size 1 1)
+					(thickness 0.15)
+				)
+			)
+		)
+		(attr smd)
+		(duplicate_pad_numbers_are_jumpers no)
+		(fp_poly
+			(pts
+				(xy 0 0) (xy -1.5 -2) (xy 1.5 -2)
+			)
+			(stroke
+				(width 0.1)
+				(type solid)
+			)
+			(fill yes)
+			(layer "F.SilkS")
+		)
+		(embedded_fonts no)
+	)
 	(footprint "FormantKO-Panel:Switch_Mini_Toggle"
 		(layer "F.Cu")
@@
 		(embedded_fonts no)
 	)
-	(gr_poly
-		(pts
-			(xy 184.635894 95.240428) (xy 181.635894 92.240428) (xy 187.635894 92.240428)
-		)
-		(stroke
-			(width 0.1)
-			(type solid)
-		)
-		(fill yes)
-		(layer "F.SilkS")
-	)
-	(gr_poly
-		(pts
-			(xy 201.635894 61.240428) (xy 198.635894 58.240428) (xy 204.635894 58.240428)
-		)
-		(stroke
-			(width 0.1)
-			(type solid)
-		)
-		(fill yes)
-		(layer "F.SilkS")
-	)
-	(gr_poly
-		(pts
-			(xy 218.635894 95.240428) (xy 215.635894 92.240428) (xy 221.635894 92.240428)
-		)
-		(stroke
-			(width 0.1)
-			(type solid)
-		)
-		(fill yes)
-		(layer "F.SilkS")
-	)
 	(gr_rect
