File: modules/24_KRIMISIZER/KRIMISIZER.kicad_pcb (KiCad board)
At the start: 2 copper layers, 160 x 100 mm, 2 parts, among them J1 Card_Connector

Commit message: rfm work
Parts:
- added C1: 22µ, FormantKO:CP_Axial_600, F.Cu at (198.5, 89.9)
- added C2: 1µ5, FormantKO:CP_Axial_600, F.Cu at (170.6, 95.0)
- added C3: 47µ, FormantKO:CP_Axial_600, F.Cu at (150.2, 95.0)
- added C4: 470µ, FormantKO:CP_Axial_600, F.Cu at (135.0, 74.7)
- added C5: 4µ7, FormantKO:CP_Axial_600, F.Cu at (135.0, 67.1)
- added C6: 47µ, FormantKO:CP_Axial_600, F.Cu at (81.7, 84.8)
- added C7: 680n, FormantKO:C_Disc, F.Cu at (119.8, 67.1)
- added C8: 4µ7, FormantKO:CP_Axial_600, F.Cu at (91.8, 95.0)
- added D1: 1N4148, FormantKO:DUS, F.Cu at (188.3, 74.7)
- added D2: 1N4148, FormantKO:DUS, F.Cu at (173.1, 74.7)
- added D3: 1N4148, FormantKO:DUS, F.Cu at (102.0, 72.1)
- added D4: 1N4148, FormantKO:DUS, F.Cu at (96.9, 72.1)
- added P1: 470k, FormantKO:Potentiometer_Trimmer, F.Cu at (165.5, 125.5)
- added P2: 470k, FormantKO:Potentiometer_Trimmer, F.Cu at (152.8, 125.5)
- added P3: 100k, FormantKO:Potentiometer_Trimmer, F.Cu at (127.4, 125.5)
- added P4: 22k, FormantKO:Potentiometer_Trimmer, F.Cu at (140.1, 125.5)
- added P5: 4k7, FormantKO:Potentiometer_Trimmer, F.Cu at (99.4, 125.5)
- added P6: 4k7, FormantKO:Potentiometer_Trimmer, F.Cu at (113.4, 125.5)
- added R1: 2k2, FormantKO:R_Axial_Horizontal, F.Cu at (161.7, 59.4)
- added R10: 10k, FormantKO:R_Axial_Horizontal, F.Cu at (145.2, 93.7)
- added R11: 1k, FormantKO:R_Axial_Horizontal, F.Cu at (133.7, 89.9)
- added R12: 1k, FormantKO:R_Axial_Horizontal, F.Cu at (133.7, 59.4)
- added R13: 1k, FormantKO:R_Axial_Horizontal, F.Cu at (133.7, 95.0)
- added R14: 1k, FormantKO:R_Axial_Horizontal, F.Cu at (117.2, 93.7)
- added R15: 1k, FormantKO:R_Axial_Horizontal, F.Cu at (112.1, 93.7)
- added R16: 2k2, FormantKO:R_Axial_Horizontal, F.Cu at (107.1, 93.7)
- added R17: 2k2, FormantKO:R_Axial_Horizontal, F.Cu at (102.0, 93.7)
- added R18: 22k, FormantKO:R_Axial_Horizontal, F.Cu at (96.9, 93.7)
- added R19: 12k, FormantKO:R_Axial_Horizontal, F.Cu at (85.5, 128.0)
- added R2: 100k, FormantKO:R_Axial_Horizontal, F.Cu at (185.8, 93.7)
- added R20: 100k, FormantKO:R_Axial_Horizontal, F.Cu at (91.8, 73.4)
- added R3: 100k, FormantKO:R_Axial_Horizontal, F.Cu at (180.7, 93.7)
- added R4: 10k, FormantKO:R_Axial_Horizontal, F.Cu at (175.6, 93.7)
- added R5: 100k, FormantKO:R_Axial_Horizontal, F.Cu at (161.7, 64.5)
- added R6: 1k, FormantKO:R_Axial_Horizontal, F.Cu at (160.4, 93.7)
- added R7: 10k, FormantKO:R_Axial_Horizontal, F.Cu at (165.5, 93.7)
- added R8: 1k, FormantKO:R_Axial_Horizontal, F.Cu at (155.3, 93.7)
- added R9: 1k, FormantKO:R_Axial_Horizontal, F.Cu at (154.1, 74.7)
- added S1: ~, FormantKO:Panel_Connector_1x03, F.Cu at (63.9, 79.8)
- added S2: ~, FormantKO:Panel_Connector_1x03, F.Cu at (63.9, 95.0)
- added S3: ~, FormantKO:Panel_Connector_1x03, F.Cu at (63.9, 110.2)
- added T1: TUN, FormantKO:TO-18, F.Cu at (185.8, 64.5)
- added T2: TUP, FormantKO:TO-18, F.Cu at (175.6, 64.5)
- added T3: TUN, FormantKO:TO-18, F.Cu at (147.7, 62.0)
- added T4: TUN, FormantKO:TO-18, F.Cu at (109.6, 63.2)
- added T5: TUN, FormantKO:TO-18, F.Cu at (109.6, 73.4)
- added T6: TUN, FormantKO:TO-18, F.Cu at (138.8, 103.9)
- added T7: TUN, FormantKO:TO-18, F.Cu at (129.9, 102.6)
- added T8: TUN, FormantKO:TO-18, F.Cu at (89.3, 116.6)
- MH1: value ~ -> CardBracket; footprint FormantKO:Schroff_60807-011_3U_Pair -> FormantKO:Card_Bracket
- moved MH1 50.0 mm to (55.0, 95.0)
- moved J1 40.2 mm to (215.0, 95.0)
