File: modules/ADSR/system.kicad_sch (KiCad schematic)
At the start: 7 parts, among them J1 CardConnector, J2 ENV SELECT, J3 GATE SELECT, J4 EOS

Commit message: finish adsr module & panel
Other:
- company: (none) -> THE HOUSE OF GALAHAD
- title: (none) -> ADSR
Changed lines of the file:
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@@
 	(generator "eeschema")
 	(generator_version "10.0")
-	(paper "A4")
+	(paper "USLetter")
+	(title_block
+		(title "ADSR")
+		(date "2026-06-20")
+		(rev "A")
+		(company "THE HOUSE OF GALAHAD")
+		(comment 1 "FORMANT-KO")
+	)
 	(junction
 		(at 104.14 62.23)
