File: modules/ADSR/system.kicad_sch (KiCad schematic)
At the start: 7 parts, among them J1 CardConnector, J2 ENV SELECT, J3 GATE SELECT, J4 EOS

Commit message: sequencer work
Parts:
- added J5: EGATE, FormantKO:PanelConnector_1x03, symbol FormantKO:MonoJack_Switched
Connections:
- net GATE: now also J5.1 (T); no longer J3.1 (Pin_1), J3.3 (Pin_3)
- net GND: now also J5.2 (S)
- new net IGATE: J3.1 (Pin_1), J3.3 (Pin_3), J5.3 (N)
Changed lines of the file:
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@@
 	(title_block
 		(title "ADSR")
-		(date "2026-06-20")
-		(rev "A")
+		(date "2026-07-04")
+		(rev "B")
 		(company "THE HOUSE OF GALAHAD")
 		(comment 1 "FORMANT-KO")
@@
 	(wire
 		(pts
+			(xy 152.4 116.84) (xy 160.02 116.84)
+		)
+		(stroke
+			(width 0)
+			(type default)
+		)
+	)
+	(wire
+		(pts
+			(xy 152.4 119.38) (xy 160.02 119.38)
+		)
+		(stroke
+			(width 0)
+			(type default)
+		)
+	)
+	(wire
+		(pts
 			(xy 177.8 58.42) (xy 177.8 63.5)
 		)
@@
 			(width 0)
 			(type default)
+		)
+	)
+	(global_label "GATE"
+		(shape output)
+		(at 152.4 119.38 180)
+		(fields_autoplaced yes)
+		(effects
+			(font
+				(size 1.27 1.27)
+			)
+			(justify right)
+		)
+		(property "Intersheetrefs" "${INTERSHEET_REFS}"
+			(at 144.8445 119.38 0)
+			(hide yes)
+			(show_name no)
+			(do_not_autoplace no)
+			(effects
+				(font
+					(size 1.27 1.27)
+				)
+				(justify right)
+			)
 		)
 	)
@@
 		)
 	)
+	(global_label "IGATE"
+		(shape input)
+		(at 152.4 116.84 180)
+		(fields_autoplaced yes)
+		(effects
+			(font
+				(size 1.27 1.27)
+			)
+			(justify right)
+		)
+		(property "Intersheetrefs" "${INTERSHEET_REFS}"
+			(at 144.2397 116.84 0)
+			(hide yes)
+			(show_name no)
+			(do_not_autoplace no)
+			(effects
+				(font
+					(size 1.27 1.27)
+				)
+				(justify right)
+			)
+		)
+	)
 	(global_label "GATE1"
 		(shape input)
@@
 		)
 	)
-	(global_label "GATE"
+	(global_label "IGATE"
 		(shape output)
 		(at 99.06 102.87 180)
@@
 		)
 		(property "Intersheetrefs" "${INTERSHEET_REFS}"
-			(at 91.5045 102.87 0)
+			(at 90.8997 102.87 0)
 			(hide yes)
 			(show_name no)
@@
 	)
 	(symbol
+		(lib_id "FormantKO:MonoJack_Switched")
+		(at 165.1 119.38 180)
+		(unit 1)
+		(body_style 1)
+		(exclude_from_sim no)
+		(in_bom yes)
+		(on_board yes)
+		(in_pos_files yes)
+		(dnp no)
+		(fields_autoplaced yes)
+		(property "Reference" "J5"
+			(at 170.18 117.4749 0)
+			(show_name no)
+			(do_not_autoplace no)
+			(effects
+				(font
+					(size 1.27 1.27)
+				)
+				(justify right)
+			)
+		)
+		(property "Value" "EGATE"
+			(at 170.18 120.0149 0)
+			(show_name no)
+			(do_not_autoplace no)
+			(effects
+				(font
+					(size 1.27 1.27)
+				)
+				(justify right)
+			)
+		)
+		(property "Footprint" "FormantKO:PanelConnector_1x03"
+			(at 165.1 119.38 0)
+			(hide yes)
+			(show_name no)
+			(do_not_autoplace no)
+			(effects
+				(font
+					(size 1.27 1.27)
+				)
+			)
+		)
+		(property "Datasheet" ""
+			(at 165.1 119.38 0)
+			(hide yes)
+			(show_name no)
+			(do_not_autoplace no)
+			(effects
+				(font
+					(size 1.27 1.27)
+				)
+			)
+		)
+		(property "Description" "Audio Jack, 2 Poles (Mono / TS), Switched T Pole (Normalling)"
+			(at 165.1 119.38 0)
+			(hide yes)
+			(show_name no)
+			(do_not_autoplace no)
+			(effects
+				(font
+					(size 1.27 1.27)
+				)
+			)
+		)
+		(pin "3"
+		)
+		(pin "1"
+		)
+		(pin "2"
+		)
+		(instances
+			(project "ADSR"
+				(path "/d2c8cc99-9c9f-481f-b15d-dad87d2b88db"
+					(reference "J5")
+					(unit 1)
+				)
+			)
+		)
+	)
+	(symbol
 		(lib_id "power:-15V")
 		(at 177.8 76.2 180)
@@
 					(unit 1)
 				)
+			)
+		)
+	)
+	(symbol
+		(lib_id "power:GND")
+		(at 160.02 121.92 0)
+		(unit 1)
+		(body_style 1)
+		(exclude_from_sim no)
+		(in_bom yes)
+		(on_board yes)
+		(in_pos_files yes)
+		(dnp no)
+		(property "Reference" "#PWR010"
+			(at 160.02 128.27 0)
+			(hide yes)
+			(show_name no)
+			(do_not_autoplace no)
+			(effects
+				(font
+					(size 1.27 1.27)
+				)
+			)
+		)
+		(property "Value" "GND"
+			(at 160.02 125.73 0)
+			(show_name no)
+			(do_not_autoplace no)
+			(effects
+				(font
+					(size 1.27 1.27)
+				)
+			)
+		)
+		(property "Footprint" ""
+			(at 160.02 121.92 0)
+			(hide yes)
+			(show_name no)
+			(do_not_autoplace no)
+			(effects
+				(font
+					(size 1.27 1.27)
+				)
+			)
+		)
+		(property "Datasheet" ""
+			(at 160.02 121.92 0)
+			(hide yes)
+			(show_name no)
+			(do_not_autoplace no)
+			(effects
+				(font
+					(size 1.27 1.27)
+				)
+			)
+		)
+		(property "Description" "Power symbol creates a global label with name \"GND\" , ground"
+			(at 160.02 121.92 0)
+			(hide yes)
+			(show_name no)
+			(do_not_autoplace no)
+			(effects
+				(font
+					(size 1.27 1.27)
+				)
+			)
+		)
+		(pin "1"
+		)
+		(instances
+			(project "ADSR"
+				(path "/d2c8cc99-9c9f-481f-b15d-dad87d2b88db"
+					(reference "#PWR010")
+					(unit 1)
+				)

Commit message: adsr additions
Parts:
- added J6: NO EGATE, FormantKO:Jumper_1x02, symbol FormantKO:Jumper_1x02
Connections:
- net GATE: now also J6.2 (Pin_2)
- net IGATE: now also J6.1 (Pin_1)
Changed lines of the file:
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@@
+		)
+	)
+	(global_label "GATE"
+		(shape output)
+		(at 161.29 137.16 180)
+		(fields_autoplaced yes)
+		(effects
+			(font
+				(size 1.27 1.27)
+			)
+			(justify right)
+		)
+		(property "Intersheetrefs" "${INTERSHEET_REFS}"
+			(at 153.7345 137.16 0)
+			(hide yes)
+			(show_name no)
+			(do_not_autoplace no)
+			(effects
+				(font
+					(size 1.27 1.27)
+				)
+				(justify right)
+			)
 		)
 	)
@@
 				)
 				(justify left)
+			)
+		)
+	)
+	(global_label "IGATE"
+		(shape input)
+		(at 161.29 134.62 180)
+		(fields_autoplaced yes)
+		(effects
+			(font
+				(size 1.27 1.27)
+			)
+			(justify right)
+		)
+		(property "Intersheetrefs" "${INTERSHEET_REFS}"
+			(at 153.1297 134.62 0)
+			(hide yes)
+			(show_name no)
+			(do_not_autoplace no)
+			(effects
+				(font
+					(size 1.27 1.27)
+				)
+				(justify right)
 			)
 		)
@@
 			)
 		)
+	)
+	(symbol
+		(lib_id "FormantKO:Jumper_1x02")
+		(at 166.37 134.62 0)
+		(mirror y)
+		(unit 1)
+		(body_style 1)
+		(exclude_from_sim no)
+		(in_bom yes)
+		(on_board yes)
+		(in_pos_files yes)
+		(dnp no)
+		(fields_autoplaced yes)
+		(property "Reference" "J6"
+			(at 165.735 129.54 0)
+			(show_name no)
+			(do_not_autoplace no)
+			(effects
+				(font
+					(size 1.27 1.27)
+				)
+			)
+		)
+		(property "Value" "NO EGATE"
+			(at 165.735 132.08 0)
+			(show_name no)
+			(do_not_autoplace no)
+			(effects
+				(font
+					(size 1.27 1.27)
+				)
+			)
+		)
+		(property "Footprint" "FormantKO:Jumper_1x02"
+			(at 166.37 134.62 0)
+			(hide yes)
+			(show_name no)
+			(do_not_autoplace no)
+			(effects
+				(font
+					(size 1.27 1.27)
+				)
+			)
+		)
+		(property "Datasheet" ""
+			(at 166.37 134.62 0)
+			(hide yes)
+			(show_name no)
+			(do_not_autoplace no)
+			(effects
+				(font
+					(size 1.27 1.27)
+				)
+			)
+		)
+		(property "Description" "Generic connector, single row, 01x02, script generated"
+			(at 166.37 134.62 0)
+			(hide yes)
+			(show_name no)
+			(do_not_autoplace no)
+			(effects
+				(font
+					(size 1.27 1.27)
+				)
+			)
+		)
+		(pin "1"
+		)
+		(pin "2"
+		)
+		(instances
+			(project "ADSR"
+				(path "/d2c8cc99-9c9f-481f-b15d-dad87d2b88db"
+					(reference "J6")
+					(unit 1)
+				)
+			)
+		)

Commit message: adsr revisions
Parts:
- added J7: GND, FormantKO:Wire_1x01_General, symbol FormantKO:WireConnector
- C3: footprint FormantKO:CP_Axial_600 -> FormantKO:CP_Axial_700-900mil_PinSwap
- C4: footprint FormantKO:CP_Axial_600 -> FormantKO:CP_Axial_700-900mil
- J1: footprint FormantKO:Card_Connector -> FormantKO:CardConnector
- J2: footprint Connector_PinHeader_2.54mm:PinHeader_2x04_P2.54mm_Vertical -> (none)
- J3: footprint Connector_PinHeader_2.54mm:PinHeader_2x02_P2.54mm_Vertical -> (none)
- J4: footprint FormantKO:Panel_Connector_1x02 -> FormantKO:PanelConnector_1x02; Legend LEGEND -> EOS
- J5: value EGATE -> EXT GATE; Legend (none) -> EXT GATE
- J6: value NO EGATE -> NO EXT GATE
- MH1: footprint FormantKO:Card_Bracket -> FormantKO:CardBracket
Connections:
- net GND: now also J7.1
Other:
- note added: "WIRE PADS"
- moved on the sheet: C3, C4, J1, J2, J3, J4, J5, J6, MH1
