File: modules/ADSR/ADSR.kicad_sch (KiCad schematic)
At the start: 53 parts, among them IC1 µA741C, IC2 µA741C, IC3 µA741C, IC4 µA741C, IC5 µA741C, P1 1M, P2 1M, P3 1M, P4 10k, P5 25k, T1 TUN, T2 TUN, T3 TUN, T4 TUN, T5 TUN, T6 TUN

Commit message: lfos overhaul to current template
Parts:
- removed T1, T2, T3, T4, T5, T6: TUN, FormantKO:TO-18, symbol FormantKO:T_Universial_NPN
- added T1, T2, T3, T4, T5, T6: BC548C, FormantKO:TO-92, symbol FormantKO:BC548C
Connections:
- net GND: now also T1.3 (E), T2.3 (E), T4.3 (E), T5.3 (E)
- net at IC1.6, P1.2, P1.3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: now also T3.1 (C)
- net at R11.1, R6.1, R7.2: now also T2.1 (C)
- net at R5.2, R6.2: now also T1.2 (B)
- net at R11.2, R16.2: now also T5.2 (B)
- net at IC2.2 (-), IC2.6: now also T6.3 (E)
- net at R20.1: now also T6.2 (B)
- net at P3.2, P3.3: now also T6.1 (C)
- net at C1.2, R3.1: now also T1.1 (C)
- net at R18.2, R19.1, R20.2: now also T5.1 (C)
- net at P2.2, P2.3: now also T3.3 (E)
- net at R14.1: now also T3.2 (B)
- net at R14.2, R15.1, R16.1: now also T4.1 (C)
- net at C1.1, R4.1: now also T2.2 (B)
- net at R18.1, R22.2: now also T4.2 (B)

Commit message: adsr revisions
Parts:
- added J10: P1.2, FormantKO:Wire_1x01_General, symbol FormantKO:WireConnector
- added J11: P2.3, FormantKO:Wire_1x01_General, symbol FormantKO:WireConnector
- added J12: P2.2, FormantKO:Wire_1x01_General, symbol FormantKO:WireConnector
- added J13: P2.1, FormantKO:Wire_1x01_General, symbol FormantKO:WireConnector
- added J14: P3.1, FormantKO:Wire_1x01_General, symbol FormantKO:WireConnector
- added J15: P3.3, FormantKO:Wire_1x01_General, symbol FormantKO:WireConnector
- added J16: P3.2, FormantKO:Wire_1x01_General, symbol FormantKO:WireConnector
- added J17: P4.1, FormantKO:Wire_1x01_General, symbol FormantKO:WireConnector
- added J18: P4.2, FormantKO:Wire_1x01_General, symbol FormantKO:WireConnector
- added J19: P4.3, FormantKO:Wire_1x01_General, symbol FormantKO:WireConnector
- added J20: S1a, FormantKO:Wire_1x01_General, symbol FormantKO:WireConnector
- added J21: S1b, FormantKO:Wire_1x01_General, symbol FormantKO:WireConnector
- added J22: S1m, FormantKO:Wire_1x01_General, symbol FormantKO:WireConnector
- added J23: D6a, FormantKO:Wire_1x01_General, symbol FormantKO:WireConnector
- added J24: D6k, FormantKO:Wire_1x01_General, symbol FormantKO:WireConnector
- added J25: EOS, FormantKO:Wire_1x01_General, symbol FormantKO:WireConnector
- added J26: GND, FormantKO:Wire_1x01_General, symbol FormantKO:WireConnector
- added J8: P1.1, FormantKO:Wire_1x01_General, symbol FormantKO:WireConnector
- added J9: P1.3, FormantKO:Wire_1x01_General, symbol FormantKO:WireConnector
- C1: footprint FormantKO:C_Disc_300_400 -> FormantKO:C_Rect
- D1, D2, D3, D4, D5: value DUS -> 1N4148; footprint FormantKO:DUS -> FormantKO:DO-35_400mil; symbol FormantKO:D_UniversalSilicon -> FormantKO:1N4148
- D6: footprint FormantKO:Panel_Connector_1x02 -> FormantKO:PanelConnector_1x02_PinSwap; Legend (none) -> ENV IND
- D7: value DUS -> 1N4148; footprint FormantKO:DUS_500 -> FormantKO:DO-35_500mil; symbol FormantKO:D_UniversalSilicon -> FormantKO:1N4148
- P1, P2, P3: footprint FormantKO:Panel_Connector_1x03 -> FormantKO:PanelConnector_1x03
- P4: footprint FormantKO:Panel_Connector_1x03 -> FormantKO:PanelConnector_1x03_PinSwap
- P5: footprint FormantKO:Potentiometer_Trimmer -> FormantKO:Potentiometer_Trimmer_PinSwap
- R23, R24: value 27k -> 10k
- S1: footprint FormantKO:Panel_Connector_1x03 -> FormantKO:PanelConnector_1x03_PinSwap; Legend (none) -> MODE
- T1, T2, T3, T4, T5, T6: value BC548C -> BC108C; footprint FormantKO:TO-92 -> FormantKO:TO-18_Wide; symbol FormantKO:BC548C -> FormantKO:BC108C
Connections:
- net EOS: now also J25.1
- net GATE: now also J21.1
- net GND: now also T1.1 (E), T2.1 (E), T4.1 (E), T5.1 (E), J17.1, J26.1; no longer T1.3 (E), T2.3 (E), T4.3 (E), T5.3 (E)
- net at D5.1 (K), D6.2 (A), IC5.2 (-)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: now also J23.1
- net at D5.2 (A), D6.1 (K), IC5.6: now also J24.1
- net at R11.1, R6.1, R7.2: now also T2.3 (C); no longer T2.1 (C)
- net at IC1.6, P1.2, P1.3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: now also T3.3 (C), J10.1, J9.1; no longer T3.1 (C)
- net at P2.2, P2.3: now also T3.1 (E), J11.1, J12.1; no longer T3.3 (E)
- net at P3.1, R21.2: now also J14.1
- net at P3.2, P3.3: now also T6.3 (C), J15.1, J16.1; no longer T6.1 (C)
- net at IC2.2 (-), IC2.6: now also T6.1 (E); no longer T6.3 (E)
- net at R1.1, R2.2, S1.1 (a): now also J20.1
- net at C1.2, R3.1: now also T1.3 (C); no longer T1.1 (C)
- net at R18.2, R19.1, R20.2: now also T5.3 (C); no longer T5.1 (C)
- net at IC1.3 (+), R8.1, S1.2 (c): now also J22.1
- net at IC2.3 (+), P4.2: now also J18.1
- net at P2.1, R17.2: now also J13.1
- net at R14.2, R15.1, R16.1: now also T4.3 (C); no longer T4.1 (C)
- net at P4.3, P5.1, P5.2: now also J19.1
- net at P1.1, R13.2: now also J8.1
