File: modules/VCO/system.kicad_sch (KiCad schematic)
At the start: 14 parts, among them J1 Card_Connector, J2 KOV SELECT, J3 IOS SELECT, J5 Mono_Jack, J6 Mono_Jack, J7 Mono_Jack, J8 Mono_Jack

Commit message: vco pcb work
Parts:
- added IC1: 7413, FormantKO:DIP-14, symbol FormantKO:7413
- C10, C11: footprint FormantKO:CP_Axial_600 -> FormantKO:CP_Axial_1000
- C3, C4, C5: footprint FormantKO:C_Disc -> FormantKO:C_Rect
- J1: footprint FormantKO:Card_Connector -> FormantKO:CardConnector; symbol FormantKO:Card_Connector -> FormantKO:CardConnector
- J5: value Mono_Jack -> FM; footprint FormantKO:Panel_Connector_1x02 -> FormantKO:PanelConnector_1x02; symbol FormantKO:Mono_Jack -> FormantKO:MonoJack; Legend FM -> (none)
- J6: value Mono_Jack -> ECV; footprint FormantKO:Panel_Connector_1x02 -> FormantKO:PanelConnector_1x02; symbol FormantKO:Mono_Jack -> FormantKO:MonoJack; Legend ECV -> (none)
- J7: value Mono_Jack -> PWM; footprint FormantKO:Panel_Connector_1x02 -> FormantKO:PanelConnector_1x02; symbol FormantKO:Mono_Jack -> FormantKO:MonoJack; Legend PWM -> (none)
- J8: value Mono_Jack -> EOS; footprint FormantKO:Panel_Connector_1x02 -> FormantKO:PanelConnector_1x02; symbol FormantKO:Mono_Jack -> FormantKO:MonoJack; Legend EOS -> (none)
- MH1, MH2: footprint FormantKO:Card_Bracket -> FormantKO:CardBracket; symbol FormantKO:Card_Bracket -> FormantKO:CardBracket
Connections:
- net +5V: now also IC1.14 (V_{cc})
- net GND: now also IC1.7 (GND)
- no-connect marks 13 -> 18

Commit message: vco pcb work
Parts:
- C3, C4, C5: footprint FormantKO:C_Rect -> FormantKO:C_Rect_300
Changed lines of the file:
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@@
 			)
 		)
-		(property "Footprint" "FormantKO:C_Rect"
+		(property "Footprint" "FormantKO:C_Rect_300"
 			(at 63.5 165.1 0)
 			(hide yes)
@@
 			)
 		)
-		(property "Footprint" "FormantKO:C_Rect"
+		(property "Footprint" "FormantKO:C_Rect_300"
 			(at 50.8 165.1 0)
 			(hide yes)
@@
 			)
 		)
-		(property "Footprint" "FormantKO:C_Rect"
+		(property "Footprint" "FormantKO:C_Rect_300"
 			(at 63.5 177.8 0)
 			(hide yes)
