File: system/VALIDATOR_JIG/VALIDATOR_JIG.kicad_sch (KiCad schematic)
At the start: 15 parts, among them IC1 µA726, J1 POWER

Commit message: 726 tester updates
Parts:
- added TP5: GND, FormantKO:KEYSTONE_5001, symbol FormantKO:TestPoint
- TP1, TP3: footprint FormantKO:KEYSTONE_5005 -> FormantKO:KEYSTONE_5000
- TP2, TP4: footprint FormantKO:KEYSTONE_5001 -> FormantKO:KEYSTONE_5117
Connections:
- net GND: now also TP5.1
Changed lines of the file:
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@@
+	)
+	(junction
+		(at 153.67 88.9)
+		(diameter 0)
+		(color 0 0 0 0)
 	)
 	(junction
@@
 	(wire
 		(pts
-			(xy 149.86 88.9) (xy 158.75 88.9)
+			(xy 149.86 88.9) (xy 153.67 88.9)
 		)
 		(stroke
@@
 		(pts
 			(xy 142.24 73.66) (xy 142.24 77.47)
+		)
+		(stroke
+			(width 0)
+			(type default)
+		)
+	)
+	(wire
+		(pts
+			(xy 153.67 88.9) (xy 158.75 88.9)
 		)
 		(stroke
@@
 			)
 		)
-		(property "Footprint" "FormantKO:KEYSTONE_5005"
+		(property "Footprint" "FormantKO:KEYSTONE_5000"
 			(at 142.24 77.47 0)
 			(hide yes)
@@
 			)
 		)
-		(property "Footprint" "FormantKO:KEYSTONE_5001"
+		(property "Footprint" "FormantKO:KEYSTONE_5117"
 			(at 142.24 100.33 0)
 			(hide yes)
@@
 			)
 		)
-		(property "Footprint" "FormantKO:KEYSTONE_5005"
+		(property "Footprint" "FormantKO:KEYSTONE_5000"
 			(at 147.32 77.47 0)
 			(hide yes)
@@
 	)
 	(symbol
+		(lib_id "FormantKO:TestPoint")
+		(at 153.67 88.9 0)
+		(unit 1)
+		(body_style 1)
+		(exclude_from_sim no)
+		(in_bom yes)
+		(on_board yes)
+		(in_pos_files yes)
+		(dnp no)
+		(property "Reference" "TP5"
+			(at 153.67 87.63 0)
+			(show_name no)
+			(do_not_autoplace no)
+			(effects
+				(font
+					(size 1.27 1.27)
+				)
+				(justify bottom)
+			)
+		)
+		(property "Value" "GND"
+			(at 153.67 90.17 0)
+			(show_name no)
+			(do_not_autoplace no)
+			(effects
+				(font
+					(size 1.27 1.27)
+				)
+				(justify top)
+			)
+		)
+		(property "Footprint" "FormantKO:KEYSTONE_5001"
+			(at 158.75 88.9 0)
+			(hide yes)
+			(show_name no)
+			(do_not_autoplace no)
+			(effects
+				(font
+					(size 1.27 1.27)
+				)
+			)
+		)
+		(property "Datasheet" ""
+			(at 158.75 88.9 0)
+			(hide yes)
+			(show_name no)
+			(do_not_autoplace no)
+			(effects
+				(font
+					(size 1.27 1.27)
+				)
+			)
+		)
+		(property "Description" "test point"
+			(at 153.67 88.9 0)
+			(hide yes)
+			(show_name no)
+			(do_not_autoplace no)
+			(effects
+				(font
+					(size 1.27 1.27)
+				)
+			)
+		)
+		(pin "1"
+		)
+		(instances
+			(project "VALIDATOR_JIG"
+				(path "/edaf0cb6-2af4-45d1-ac73-5a13d9505154"
+					(reference "TP5")
+					(unit 1)
+				)
+			)
+		)
+	)
+	(symbol
 		(lib_id "FormantKO:µA726")
 		(at 139.7 88.9 0)
@@
 			)
 		)
-		(property "Footprint" "FormantKO:KEYSTONE_5001"
+		(property "Footprint" "FormantKO:KEYSTONE_5117"
 			(at 147.32 100.33 0)
 			(hide yes)
