File: modules/VCF_12/VCF_12.kicad_pcb (KiCad board)
At the start: 2 copper layers, 160 x 200 mm, 5 parts, among them J1 BUS CONNECTOR

Commit message: vcf work
Parts:
- added C1: 680n, FormantKO:C_Disc, F.Cu at (61.8, 114.8)
- added C10: 680n, FormantKO:C_Disc, F.Cu at (49.1, 145.3)
- added C2: 1n, FormantKO:C_Disc, F.Cu at (131.7, 117.0)
- added C3: C, FormantKO:C_Disc, F.Cu at (158.3, 125.0)
- added C4: C, FormantKO:C_Disc, F.Cu at (168.5, 117.4)
- added C5: C, FormantKO:C_Disc, F.Cu at (66.9, 163.1)
- added C6: 33p, FormantKO:C_Disc, F.Cu at (145.6, 158.0)
- added C7: 33p, FormantKO:C_Disc, F.Cu at (135.5, 173.3)
- added C8: 180p, FormantKO:C_Disc, F.Cu at (117.7, 140.2)
- added C9: 180p, FormantKO:C_Disc, F.Cu at (84.7, 150.4)
- added IC1: CA3084, FormantKO:DIP-14, F.Cu at (86.9, 98.7)
- added IC2: µA741C, FormantKO:DIP-8, F.Cu at (130.4, 106.2)
- added IC3: µA741C, FormantKO:DIP-8, F.Cu at (159.6, 172.0)
- added IC4: CA3080, FormantKO:DIP-8, F.Cu at (126.6, 161.8)
- added IC5: CA3080, FormantKO:DIP-8, F.Cu at (93.6, 161.8)
- added IC6: µA741C, FormantKO:DIP-8, F.Cu at (68.2, 131.3)
- added J2: TM, FormantKO:Panel_Connector_1x02, F.Cu at (31.3, 80.5)
- added J3: ECV, FormantKO:Panel_Connector_1x02, F.Cu at (31.3, 65.3)
- added J4: ES, FormantKO:Panel_Connector_1x02, F.Cu at (31.3, 169.5)
- added J5: EOS, FormantKO:Panel_Connector_1x02, F.Cu at (31.3, 154.2)
- added P1: 100k, FormantKO:Panel_Connector_1x03, F.Cu at (31.3, 104.7)
- added P2: 47k, FormantKO:Panel_Connector_1x03, F.Cu at (31.3, 92.0)
- added P3: 47k, FormantKO:Panel_Connector_1x03, F.Cu at (44.0, 79.3)
- added P4: 47k, FormantKO:Panel_Connector_1x03, F.Cu at (44.0, 168.3)
- added P5: 100k, FormantKO:Panel_Connector_1x03, F.Cu at (31.3, 180.9)
- added P6: 4k7, FormantKO:Panel_Connector_1x03, F.Cu at (44.0, 155.4)
- added P7: 100k, FormantKO:Potentiometer_Trimmer, F.Cu at (97.4, 117.4)
- added P8: 500R, FormantKO:Potentiometer_Trimmer, F.Cu at (105.8, 95.0)
- added R1: 100k, FormantKO:R_Axial_Horizontal, F.Cu at (65.6, 109.8)
- added R10: 27k, FormantKO:R_Axial_Horizontal, F.Cu at (125.3, 136.4)
- added R11: 39k, FormantKO:R_Axial_Horizontal, F.Cu at (145.6, 172.0)
- added R12: 39k, FormantKO:R_Axial_Horizontal, F.Cu at (158.3, 156.8)
- added R13: 39k, FormantKO:R_Axial_Horizontal, F.Cu at (163.4, 156.8)
- added R14: 39k, FormantKO:R_Axial_Horizontal, F.Cu at (168.5, 156.8)
- added R15: 39k, FormantKO:R_Axial_Horizontal, F.Cu at (150.7, 156.8)
- added R16: 39k, FormantKO:R_Axial_Horizontal, F.Cu at (168.5, 172.0)
- added R17: 8k2, FormantKO:R_Axial_Horizontal, F.Cu at (145.6, 139.0)
- added R18: 27k, FormantKO:R_Axial_Horizontal, F.Cu at (150.7, 172.0)
- added R19: 1k, FormantKO:R_Axial_Horizontal, F.Cu at (47.9, 180.9)
- added R2: 100k, FormantKO:R_Axial_Horizontal, F.Cu at (80.3, 113.8)
- added R20: 39k, FormantKO:R_Axial_Horizontal, F.Cu at (140.6, 156.8)
- added R21: 100R, FormantKO:R_Axial_Horizontal, F.Cu at (140.6, 139.0)
- added R22: 100R, FormantKO:R_Axial_Horizontal, F.Cu at (135.5, 156.8)
- added R23: 12k, FormantKO:R_Axial_Horizontal, F.Cu at (124.0, 170.7)
- added R24: 39k, FormantKO:R_Axial_Horizontal, F.Cu at (102.5, 164.4)
- added R25: 100R, FormantKO:R_Axial_Horizontal, F.Cu at (102.5, 149.1)
- added R26: 100R, FormantKO:R_Axial_Horizontal, F.Cu at (107.5, 149.1)
- added R27: 12k, FormantKO:R_Axial_Horizontal, F.Cu at (83.4, 170.7)
- added R28: 100k, FormantKO:R_Axial_Horizontal, F.Cu at (52.9, 135.2)
- added R29: 100k, FormantKO:R_Axial_Horizontal, F.Cu at (52.9, 130.1)
- added R3: 100k, FormantKO:R_Axial_Horizontal, F.Cu at (65.6, 94.8)
- added R30: 100k, FormantKO:R_Axial_Horizontal, F.Cu at (52.9, 125.0)
- added R31: 33k, FormantKO:R_Axial_Horizontal, F.Cu at (70.7, 122.5)
- added R32: 470R, FormantKO:R_Axial_Horizontal, F.Cu at (63.1, 147.9)
- added R33: 27k, FormantKO:R_Axial_Horizontal, F.Cu at (89.8, 146.6)
- added R34: 100k, FormantKO:R_Axial_Horizontal, F.Cu at (65.6, 140.2)
- added R4: 33k, FormantKO:R_Axial_Horizontal, F.Cu at (65.6, 104.8)
- added R5: 47k, FormantKO:R_Axial_Horizontal, F.Cu at (65.6, 99.8)
- added R6: 1k8, FormantKO:R_Axial_Horizontal, F.Cu at (114.2, 111.7)
- added R7: 330k, FormantKO:R_Axial_Horizontal, F.Cu at (119.2, 106.3)
- added R8: 2k2, FormantKO:R_Axial_Horizontal, F.Cu at (96.6, 108.0)
- added R9: 330k, FormantKO:R_Axial_Horizontal, F.Cu at (152.2, 113.3)
- added S1: ECV/KOV, FormantKO:Panel_Connector_1x03, F.Cu at (44.0, 66.5)
- added S2: HP, FormantKO:Panel_Connector_1x03, F.Cu at (31.3, 142.8)
- added S3: BP, FormantKO:Panel_Connector_1x03, F.Cu at (31.3, 130.1)
- added S4: LP, FormantKO:Panel_Connector_1x03, F.Cu at (31.3, 117.4)
- added T1: N-FET, FormantKO:TO-92, F.Cu at (117.7, 160.6)
- added T2: N-FET, FormantKO:TO-92, F.Cu at (84.7, 160.6)
- J1: value BUS CONNECTOR -> DIN_Male
Connections:
- J1 pad A1: unconnected-(J1-PadA1) -> KOV
- J1 pad A10: unconnected-(J1-PadA10) -> +15V
- J1 pad A11: unconnected-(J1-PadA11) -> VCO3
- J1 pad A12: unconnected-(J1-PadA12) -> VCO3
- J1 pad A13: unconnected-(J1-PadA13) -> VCO2
- J1 pad A14: unconnected-(J1-PadA14) -> VCO1
- J1 pad A15: unconnected-(J1-PadA15) -> VCO1
- J1 pad A16: unconnected-(J1-PadA16) -> IOS
- J1 pad A2: unconnected-(J1-PadA2) -> KOV
- J1 pad A3: unconnected-(J1-PadA3) -> ENV
- J1 pad A4: unconnected-(J1-PadA4) -> ENV
- J1 pad A5: unconnected-(J1-PadA5) -> -15V
- J1 pad A6: unconnected-(J1-PadA6) -> -15V
- J1 pad A7: unconnected-(J1-PadA7) -> GND
- J1 pad A8: unconnected-(J1-PadA8) -> GND
- J1 pad A9: unconnected-(J1-PadA9) -> +15V
- J1 pad B1: unconnected-(J1-PadB1) -> KOV
- J1 pad B10: unconnected-(J1-PadB10) -> +15V
- J1 pad B11: unconnected-(J1-PadB11) -> VCO3
- J1 pad B12: unconnected-(J1-PadB12) -> VCO2
- J1 pad B13: unconnected-(J1-PadB13) -> VCO2
- J1 pad B14: unconnected-(J1-PadB14) -> VCO1
- J1 pad B15: unconnected-(J1-PadB15) -> IOS
- J1 pad B16: unconnected-(J1-PadB16) -> IOS
- J1 pad B2: unconnected-(J1-PadB2) -> KOV
- J1 pad B3: unconnected-(J1-PadB3) -> ENV
- J1 pad B4: unconnected-(J1-PadB4) -> ENV
- J1 pad B5: unconnected-(J1-PadB5) -> -15V
- J1 pad B6: unconnected-(J1-PadB6) -> -15V
- J1 pad B7: unconnected-(J1-PadB7) -> GND
- J1 pad B9: unconnected-(J1-PadB9) -> +15V
Other:
- board text removed: "INCOMPLETE"

Commit message: vcf_12 pcb layout
Parts:
- removed H1, H2, H3, H4: MountingHole, FormantKO:MountingHole_2.7mm_M2.5
- added J6: EOS, FormantKO:PanelConnector_1x02, F.Cu at (31.3, 178.9)
- added MH1: CardBracket, FormantKO:CardBracket, F.Cu at (25.0, 197.6)
- added MH2: CardBracket, FormantKO:CardBracket, F.Cu at (25.0, 64.2)
- C1, C10, C2, C5: footprint FormantKO:C_Disc -> FormantKO:C_Rect
- C3, C4: value C -> 680n; footprint FormantKO:C_Disc -> FormantKO:C_Rect
- C6, C7, C8, C9: footprint FormantKO:C_Disc -> FormantKO:C_Rect_200
- J1: value DIN_Male -> CardConnector; footprint FormantKO:DIN_Male -> FormantKO:CardConnector
- J2: value TM -> KOV SELECT; footprint FormantKO:Panel_Connector_1x02 -> Connector_PinHeader_2.54mm:PinHeader_2x02_P2.54mm_Vertical
- J3: value ECV -> ENV SELECT; footprint FormantKO:Panel_Connector_1x02 -> Connector_PinHeader_2.54mm:PinHeader_2x04_P2.54mm_Vertical
- J4: value ES -> IOS SELECT; footprint FormantKO:Panel_Connector_1x02 -> Connector_PinHeader_2.54mm:PinHeader_2x02_P2.54mm_Vertical
- J5: value EOS -> ES; footprint FormantKO:Panel_Connector_1x02 -> FormantKO:PanelConnector_1x02
- P1, P2, P3, P4, P5, P6, S1, S2, S3, S4: footprint FormantKO:Panel_Connector_1x03 -> FormantKO:PanelConnector_1x03
- moved J3 172.7 mm to (168.5, 170.2), turned to 0 degrees
- moved J2 159.2 mm to (168.5, 161.3), turned to 0 degrees
- moved J4 116.6 mm to (127.9, 234.9), turned to 0 degrees
- moved S1 92.3 mm to (41.5, 158.8)
- moved J1 91.9 mm to (185.0, 197.6), turned to 0 degrees
- moved P3 88.0 mm to (31.3, 166.4)
- moved S2 87.7 mm to (41.5, 229.9)
- moved S3 86.2 mm to (41.5, 215.6)
- moved S4 84.7 mm to (41.5, 201.4)
- moved P1 83.1 mm to (41.5, 187.2)
- moved P2 81.6 mm to (41.5, 173.0)
- moved R9 80.2 mm to (122.8, 187.9), turned to -90 degrees
- moved P7 72.0 mm to (92.3, 189.2)
- moved C3 71.9 mm to (155.8, 196.8)
- moved C4 71.9 mm to (171.0, 189.2)
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Connections:
- C1 pad 1: Net-(C1-Pad1) -> GND
- C1 pad 2: GND -> Net-(C1-Pad2)
- C7 pad 2: Net-(IC4--) -> Net-(IC4-+)
- J2 pad 1: GND -> KOV
- J2 pad 2: TM -> KOV1
- J3 pad 1: GND -> ENV
- J3 pad 2: ECV -> ENV1
- J4 pad 1: GND -> IOS
- J4 pad 2: ES -> VCF1
- J5 pad 2: EOS -> ES
- P1 pad 2: Net-(C1-Pad1) -> Net-(C1-Pad2)
- R1 pad 1: Net-(C1-Pad1) -> Net-(C1-Pad2)
- R20 pad 2: Net-(IC4--) -> Net-(IC4-+)
- R21 pad 2: Net-(IC4--) -> Net-(IC4-+)
- R22 pad 2: Net-(IC4-+) -> Net-(IC4--)
- R24 pad 2: Net-(IC5--) -> Net-(IC5-+)
- R25 pad 2: Net-(IC5--) -> Net-(IC5-+)
- R26 pad 2: Net-(IC5-+) -> Net-(IC5--)
Routing:
- net -15V: track 0.00 -> 45.7 mm, vias 0 -> 4
- net +15V: track 0.00 -> 38.1 mm, vias 0 -> 4
- net Net-(IC1-C): track 0.00 -> 17.8 mm, vias 0 -> 2
- net Net-(S4-a): track 0.00 -> 15.2 mm, vias 0 -> 2
- net Net-(S2-a): track 0.00 -> 12.7 mm, vias 0 -> 2
- net Net-(IC2--): track 0.00 -> 12.7 mm, vias 0 -> 2
- net GND: track 0.00 -> 12.7 mm, vias 0 -> 2
- net Net-(S3-a): track 0.00 -> 10.2 mm, vias 0 -> 2
- net (no net): track 0.00 -> 5.08 mm
- removed copper zone on B.Cu, net GND
- removed copper zone on F.Cu, net GND
Other:
- board size 160 x 200 mm -> 160 x 233.3 mm

Commit message: vcf 12 pcb
Parts:
- moved J2 5.08 mm to (168.5, 156.2)
- moved R27 5.08 mm to (93.6, 229.9)
- moved C10 3.59 mm to (51.7, 214.6)
- moved C6 2.54 mm to (148.2, 212.1)
- moved R23 2.54 mm to (124.0, 229.9)
- moved R31 2.54 mm to (75.8, 189.2)
- moved R32 2.54 mm to (65.6, 214.6)
- moved R34 2.54 mm to (65.6, 207.0)
- moved R9 2.54 mm to (120.2, 187.9)
- moved R28 2.54 mm to (52.9, 201.9)
- moved R29 2.54 mm to (52.9, 196.8)
- moved R30 2.54 mm to (52.9, 191.8)
- moved C7 2.54 mm to (140.6, 229.9)
- moved J6 1.10 mm to (31.3, 177.8)
- moved S3 1.06 mm to (41.5, 214.6)
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Routing:
- net GND: track 12.7 -> 387.9 mm, vias 2 -> 0
- net -15V: track 45.7 -> 386.9 mm, vias 4 -> 2
- net +15V: track 38.1 -> 331.8 mm, vias 4 -> 1
- net ENV: track 0.00 -> 170.5 mm
- net Net-(S2-a): track 12.7 -> 165.0 mm, vias 2 -> 0
- net Net-(S4-a): track 15.2 -> 160.1 mm, vias 2 -> 0
- net IOS: track 0.00 -> 142.0 mm
- net Net-(P5-Pad2): track 0.00 -> 139.0 mm
- net Net-(S3-a): track 10.2 -> 147.1 mm, vias 2 -> 0
- net Net-(P4-Pad2): track 0.00 -> 136.3 mm
- net KOV: track 0.00 -> 131.7 mm
- net Net-(IC1-C): track 17.8 -> 97.6 mm, vias 2 -> 0
- net VCF1: track 0.00 -> 76.1 mm
- net VCF2: track 0.00 -> 71.8 mm
- net Net-(IC1-B-Pad6): track 0.00 -> 59.5 mm
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
Commit message: vcf 12 pcb rfs
Parts:
- moved J2 1.27 mm to (168.5, 154.9)
- moved J4 0.63 mm to (127.9, 234.3)
Routing:
- net Net-(S2-a): track 165.0 -> 147.0 mm
- net Net-(S4-a): track 160.1 -> 142.0 mm
- net ENV: track 170.5 -> 156.5 mm
- net Net-(S3-a): track 147.1 -> 133.8 mm
- net +15V: track 331.8 -> 319.5 mm
- net Net-(P5-Pad2): track 139.0 -> 127.5 mm
- net -15V: track 386.9 -> 375.6 mm
- net Net-(IC1-C): track 97.6 -> 86.4 mm
- net VCF2: track 71.8 -> 62.0 mm
- net Net-(P5-Pad1): track 45.7 -> 36.2 mm
- net VCF1: track 76.1 -> 66.9 mm
- net GND: track 387.9 -> 380.5 mm
- net EOS: track 58.4 -> 51.0 mm
- net Net-(IC3-+): track 40.6 -> 34.2 mm
- net Net-(IC1-B-Pad6): track 59.5 -> 53.5 mm
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- added copper zone on B.Cu, net +15V
- added copper zone on F.Cu, net +15V
- added copper zone on B.Cu, net -15V
- added copper zone on F.Cu, net -15V
- added copper zone on B.Cu, net GND
- added copper zone on F.Cu, net GND
- added copper zone on B.Cu, net IOS
- added copper zone on B.Cu, net KOV
- added copper zone on B.Cu, net Net-(C1-Pad2)
- added copper zone on B.Cu, net Net-(C2-Pad2)
- added copper zone on B.Cu, net Net-(IC3--)
- added copper zone on B.Cu, net Net-(IC4-+)
- added copper zone on B.Cu, net Net-(IC6--)
- added copper zone on B.Cu, net Net-(P8-Pad1)
- added copper zone on F.Cu, net Net-(S2-a)
- added copper zone on B.Cu, net Net-(S3-a)
- added copper zone on F.Cu, net Net-(S4-a)
- added copper zone on B.Cu, net Net-(T1-G)
- added copper zone on B.Cu, net Net-(T2-G)
Other:
- board text added: "ENV1"
- board text added: "ENV2"
- board text added: "ENV3"
- board text added: "ENV4"
- board text added: "KOV1"
- board text added: "KOV2"
- board text added: "VCF1"
- board text added: "VCF2"
