File: modules/VCF_12/VCF_12.kicad_sch (KiCad schematic)
At the start: 0 parts

Commit message: vcf work
Parts:
- added C1, C10: 680n, FormantKO:C_Disc, symbol FormantKO:C
- added C2: 1n, FormantKO:C_Disc, symbol FormantKO:C
- added C5: C, FormantKO:C_Disc, symbol FormantKO:C
- added C6, C7: 33p, FormantKO:C_Disc, symbol FormantKO:C
- added C8, C9: 180p, FormantKO:C_Disc, symbol FormantKO:C
- added IC1: CA3084, FormantKO:DIP-14, symbol FormantKO:CA3084
- added IC2, IC3: µA741C, FormantKO:DIP-8, symbol FormantKO:Generic_OpAmp_Single
- added IC4, IC5: CA3080, FormantKO:DIP-8, symbol FormantKO:CA3080
- added IC6: µA741C, FormantKO:DIP-8, symbol FormantKO:Generic_OpAmp_Single_Swap
- added P1, P5: 100k, FormantKO:Panel_Connector_1x03, symbol FormantKO:Panel_Potentiometer_3
- added P2, P3, P4: 47k, FormantKO:Panel_Connector_1x03, symbol FormantKO:Panel_Potentiometer_3
- added P6: 4k7, FormantKO:Panel_Connector_1x03, symbol FormantKO:Panel_Potentiometer_3
- added P7: 100k, FormantKO:Potentiometer_Trimmer, symbol FormantKO:R_Trim
- added P8: 500R, FormantKO:Potentiometer_Trimmer, symbol FormantKO:R_Trim
- added R1, R2, R28, R29, R3, R30, R34: 100k, FormantKO:R_Axial_Horizontal, symbol FormantKO:R
- added R10, R18, R33: 27k, FormantKO:R_Axial_Horizontal, symbol FormantKO:R
- added R11, R12, R13, R14, R15, R16, R20, R24: 39k, FormantKO:R_Axial_Horizontal, symbol FormantKO:R
- added R17: 8k2, FormantKO:R_Axial_Horizontal, symbol FormantKO:R
- added R19: 1k, FormantKO:R_Axial_Horizontal, symbol FormantKO:R
- added R21, R22, R25, R26: 100R, FormantKO:R_Axial_Horizontal, symbol FormantKO:R
- added R23, R27: 12k, FormantKO:R_Axial_Horizontal, symbol FormantKO:R
- added R31, R4: 33k, FormantKO:R_Axial_Horizontal, symbol FormantKO:R
- added R32: 470R, FormantKO:R_Axial_Horizontal, symbol FormantKO:R
- added R5: 47k, FormantKO:R_Axial_Horizontal, symbol FormantKO:R
- added R6: 1k8, FormantKO:R_Axial_Horizontal, symbol FormantKO:R
- added R7, R9: 330k, FormantKO:R_Axial_Horizontal, symbol FormantKO:R
- added R8: 2k2, FormantKO:R_Axial_Horizontal, symbol FormantKO:R
- added S1: ECV/KOV, FormantKO:Panel_Connector_1x03, symbol FormantKO:SWITCH_SPDT
- added S2: HP, FormantKO:Panel_Connector_1x03, symbol FormantKO:SWITCH_SPDT
- added S3: BP, FormantKO:Panel_Connector_1x03, symbol FormantKO:SWITCH_SPDT
- added S4: LP, FormantKO:Panel_Connector_1x03, symbol FormantKO:SWITCH_SPDT
- added T1, T2: N-FET, FormantKO:TO-92, symbol FormantKO:N-FET
Connections:
- new net: C6.1, IC3.2 (-), R11.2, R12.2, R13.2, R14.2, R15.1, R16.1, R18.2
- new net: IC5.2 (-), R24.2, R25.2
- new net: C8.2, IC4.6, T1.1 (G)
- new net: P5.3, R23.2, R24.1, S3.1 (a), T1.2 (S)
- new net: P5.1, R19.1
- new net: P5.2, R18.1
- new net: C7.1, IC3.6, R16.2, R20.1, S2.1 (a)
- new net: C7.2, IC4.2 (-), R20.2, R21.2
- new net: P2.2, R4.1
- new net: IC1.6 (B), P8.3, R1.2, R2.2, R3.2, R4.2, R5.2
- new net: C10.2, P6.3, R32.2
- new net: C6.2, R15.2, R27.2, S4.1 (a), T2.2 (S)
- new net: R30.2, S4.2 (c)
- new net: C9.2, IC5.6, T2.1 (G)
- new net: P8.1, P8.2, R6.1
- new net: IC3.3 (+), R17.2
- new net: R3.1, S1.2 (c)
- new net: P4.2, R11.1
- new net: C5.2, P4.3
- new net: IC6.2 (-), R28.1, R29.1, R30.1, R34.1
- new net: R28.2, S2.2 (c)
- new net: C1.1, P1.2, R1.1
- new net: IC6.3 (+), R31.1
- new net: IC6.6, R32.1, R34.2
- new net: C2.1, IC1.8, IC2.2 (-), R7.1
- new net: C2.2, IC2.6, R8.2
- new net: IC1.10 (E), IC1.7 (E), R8.1
- new net: IC1.11 (C), R10.2, R33.2
- new net: R29.2, S3.2 (c)
- new net: IC4.3 (+), R22.2
- new net: IC2.3 (+), R9.1
- new net: P3.2, R5.1
- new net: IC5.3 (+), R26.2
- new net: IC5.5 (BIAS), R33.1
- new net: P7.2, R2.1
- new net: IC4.5 (BIAS), R10.1
- new net +15V: IC2.7 (V+), IC3.7 (V+), IC4.7 (V+), IC5.7 (V+), IC6.7 (V+), P1.3, T1.3 (D), T2.3 (D)
- new net -15V: IC1.4 (SUBSTRATE), IC2.4 (V-), IC3.4 (V-), IC4.4 (V-), IC5.4 (V-), IC6.4 (V-), P7.3, R23.1, R27.1, R7.2
- new net ECV: S1.3 (b)
- new net ENV: P2.3
- new net EOS: C10.1
- new net ES: C5.1
- new net GND: C1.2, C8.1, C9.1, IC1.9 (B), P1.1, P2.1, P3.3, P4.1, P6.1, P7.1, R17.1, R19.2, R21.1, R22.1, R25.1, R26.1, R31.2, R6.2, R9.2, S2.3 (b), S3.3 (b), S4.3 (b)
- new net IOS: P6.2
- new net KOV: S1.1 (a)
- new net TM: P3.1
- new net VCO1: R12.1
- new net VCO2: R13.1
- new net VCO3: R14.1
- no-connect marks 0 -> 6

Commit message: vcf_12 pcb layout
Parts:
- removed IC4, IC5: CA3080, FormantKO:DIP-8, symbol FormantKO:CA3080
- added IC4, IC5: CA3080, FormantKO:DIP-8, symbol FormantKO:CA3080_Swap
- C1, C10, C2, C5: footprint FormantKO:C_Disc -> FormantKO:C_Rect
- C6, C7, C8, C9: footprint FormantKO:C_Disc -> FormantKO:C_Rect_200
- P1, P2, P3, P4, P5, P6: footprint FormantKO:Panel_Connector_1x03 -> FormantKO:PanelConnector_1x03; symbol FormantKO:Panel_Potentiometer_3 -> FormantKO:R_Potentiometer
- P7: Legend OFFSET -> LEGEND
- P8: Legend OCTAVE/V -> LEGEND
- S1, S2, S3, S4: footprint FormantKO:Panel_Connector_1x03 -> FormantKO:PanelConnector_1x03; symbol FormantKO:SWITCH_SPDT -> FormantKO:SW_SPDT
Connections:
- net +15V: now also IC4.7 (V+), IC5.7 (V+)
- net -15V: now also IC4.4 (V-), IC5.4 (V-)
- net GND: now also C1.1; no longer C1.2
- net at R24.2, R25.2: now also IC5.3 (+)
- net at C8.2, T1.1 (G): now also IC4.6
- net at C7.2, R20.2, R21.2: now also IC4.3 (+)
- net at C9.2, T2.1 (G): now also IC5.6
- net at P1.2, R1.1: now also C1.2; no longer C1.1
- net at R22.2: now also IC4.2 (-)
- net at R26.2: now also IC5.2 (-)
- net at R33.1: now also IC5.5 (BIAS)
- net at R10.1: now also IC4.5 (BIAS)
Other:
- title: VCF_12 -> VCF-12
- moved on the sheet: C1, P5, P6

Commit message: vcf 12 pcb
Parts:
- P7: Legend LEGEND -> COARSE OFFSET
- P8: Legend LEGEND -> FREQ ADJ
Changed lines of the file:
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@@
 			)
 		)
-		(property "Legend" "LEGEND"
-			(at 81.28 46.228 0)
+		(property "Legend" "FREQ ADJ"
+			(at 69.088 45.212 0)
 			(show_name no)
 			(do_not_autoplace no)
@@
 			)
 		)
-		(property "Legend" "LEGEND"
-			(at 26.67 36.322 0)
+		(property "Legend" "COARSE OFFSET"
+			(at 41.656 40.64 0)
 			(show_name no)
 			(do_not_autoplace no)
