File: modules/VCF_24/system.kicad_sch (KiCad schematic)
At the start: 5 parts, among them J1 BUS CONNECTOR

Commit message: vcf24 work
Parts:
- added J2: ENV CONFIG, FormantKO:Jumper_1x03, symbol FormantKO:Jumper_01x03
- added J3: IOS CONFIG, FormantKO:Jumper_1x03, symbol FormantKO:Jumper_01x03
- added J4: ECV, FormantKO:Panel_Connector_1x02, symbol FormantKO:Mono_Jack
- added J5: TM, FormantKO:Panel_Connector_1x02, symbol FormantKO:Mono_Jack
- H1, H2, H3, H4: footprint FormantKO:MountingHole_2.7mm_M2.5 -> FormantKO:MountingHole_3.2mm_M3
Connections:
- net GND: now also J1.A7 (GND), J1.A8 (GND), J1.B7 (GND), J4.1 (S), J5.1 (S)
- net KOV: now reaches J1.A1 (KOV1_IN)
- net +15V: now reaches J1.A10 (+15V)
- net +15V: now also J1.A11 (+15V), J1.B10 (+15V), J1.B11 (+15V)
- net VCF1_OUT: now reaches J1.A15 (VCF1_OUT)
- net VCF1_OUT: now also J3.1 (Pin_1)
- net ENV1: now reaches J1.A2 (ENV1_IN)
- net ENV1: now also J2.1 (Pin_1)
- net -15V: now reaches J1.A5 (-15V)
- net -15V: now also J1.A6 (-15V), J1.B5 (-15V), J1.B6 (-15V)
- net VCF2_OUT: now reaches J1.B15 (VCF2_OUT)
- net VCF2_OUT: now also J3.3 (Pin_3)
- net ENV2: now reaches J1.B2 (ENV2_IN)
- net ENV2: now also J2.3 (Pin_3)
- new net ECV: J4.2 (T)
- new net ENV: J2.2 (Pin_2)
- new net IOS: J3.2 (Pin_2)
- new net TM: J5.2 (T)
- no-connect marks 31 -> 15
Other:
- moved on the sheet: H1, H2, H3, H4, J1

Commit message: restarted vcf 24 module
Parts:
- removed H1, H2, H3, H4: MountingHole, FormantKO:MountingHole_3.2mm_M3, symbol FormantKO:MountingHole
- removed J1: BUS CONNECTOR, FormantKO:DIN_Male, symbol FormantKO:DIN_Male
- removed J2: ENV CONFIG, FormantKO:Jumper_1x03, symbol FormantKO:Jumper_01x03
- removed J3: IOS CONFIG, FormantKO:Jumper_1x03, symbol FormantKO:Jumper_01x03
- removed J4: ECV, FormantKO:Panel_Connector_1x02, symbol FormantKO:Mono_Jack
- removed J5: TM, FormantKO:Panel_Connector_1x02, symbol FormantKO:Mono_Jack
- added C10, C11, C12, C13, C14, C15, C16, C17, C18: 100n, FormantKO:C_Rect, symbol FormantKO:C
- added J1: BUS CONNECTOR, FormantKO:CardConnector, symbol FormantKO:CardConnector
- added J2: KOV SELECT, Connector_PinHeader_2.54mm:PinHeader_2x02_P2.54mm_Vertical, symbol Connector_Generic:Conn_02x02_Odd_Even
- added J3: ENV SELECT, Connector_PinHeader_2.54mm:PinHeader_2x04_P2.54mm_Vertical, symbol Connector_Generic:Conn_02x04_Odd_Even
- added J4: IS_SELECT, Connector_PinHeader_2.54mm:PinHeader_2x10_P2.54mm_Vertical, symbol Connector_Generic:Conn_02x10_Odd_Even
- added J5: OS_SELECT, Connector_PinHeader_2.54mm:PinHeader_2x02_P2.54mm_Vertical, symbol Connector_Generic:Conn_02x02_Odd_Even
- added J6: ECV, FormantKO:PanelConnector_1x02, symbol FormantKO:MonoJack
- added J7: TM, FormantKO:PanelConnector_1x02, symbol FormantKO:MonoJack
- added J8: ES, FormantKO:PanelConnector_1x02, symbol FormantKO:MonoJack
- added J9: EOS, FormantKO:PanelConnector_1x02, symbol FormantKO:MonoJack
- added MH1, MH2: CardBracket, FormantKO:CardBracket, symbol FormantKO:CardBracket
Connections:
- net +15V: now also C10.1, C12.1, C14.1, C16.1, J1.a20 (+15V), J1.a22 (+15V), J1.b20 (+15V), J1.b22 (+15V)
- net -15V: now also C11.2, C13.2, C15.2, C17.2, C18.2, J1.a10 (-15V), J1.a12 (-15V), J1.b10 (-15V), J1.b12 (-15V)
- net ECV: now also J6.2 (T)
- net ENV: now also J3.1 (Pin_1), J3.3 (Pin_3), J3.5 (Pin_5), J3.7 (Pin_7)
- net ENV1: now also J1.a6 (ENV1), J3.2 (Pin_2)
- net ENV2: now also J1.b6 (ENV2), J3.4 (Pin_4)
- net GND: now also C10.2, C11.1, C12.2, C13.1, C14.2, C15.1, C16.2, C17.1, C18.1, J1.a14 (GND), J1.a16 (GND), J1.b14 (GND), J1.b16 (GND), J6.1 (S), J7.1 (S), J8.1 (S), J9.1 (S)
- net KOV: now also J2.1 (Pin_1), J2.3 (Pin_3)
- net TM: now also J7.2 (T)
- new net COM1: J1.a32 (COM1), J4.18 (Pin_18)
- new net ENV3: J1.a8 (ENV3), J3.6 (Pin_6)
- new net ENV4: J1.b8 (ENV4), J3.8 (Pin_8)
- new net EOS: J9.2 (T)
- new net ES: J8.2 (T)
- new net IS: J4.1 (Pin_1), J4.11 (Pin_11), J4.13 (Pin_13), J4.15 (Pin_15), J4.17 (Pin_17), J4.19 (Pin_19), J4.3 (Pin_3), J4.5 (Pin_5), J4.7 (Pin_7), J4.9 (Pin_9)
- new net KOV1: J1.a2 (KOV1), J2.2 (Pin_2)
- new net KOV2: J1.b2 (KOV2), J2.4 (Pin_4)
- new net OS: J5.1 (Pin_1), J5.3 (Pin_3)
- new net PA1: J1.b32 (PA1), J4.20 (Pin_20)
- new net RFM: J1.b26 (RFM), J4.8 (Pin_8)
- new net VCA1: J1.a30 (VCA1), J4.14 (Pin_14)
- new net VCA2: J1.b30 (VCA2), J4.16 (Pin_16)
- new net VCF1: J1.a28 (VCF1), J4.10 (Pin_10), J5.2 (Pin_2)
- new net VCF2: J1.b28 (VCF2), J4.12 (Pin_12), J5.4 (Pin_4)
- new net VCO1: J1.a24 (VCO1), J4.2 (Pin_2)
- new net VCO2: J1.b24 (VCO2), J4.4 (Pin_4)
- new net VCO3: J1.a26 (VCO3), J4.6 (Pin_6)
- no-connect marks 15 -> 4
Other:
- note added: "* NORMAL"
- title: VCF_24 -> TEMPLATE-6U

Commit message: vcf 24 pcb work
Parts:
- added IC2, IC5, IC8: TL074, FormantKO:DIP-14, symbol FormantKO:TL074
Connections:
- net +15V: now also IC2.4 (V+), IC5.4 (V+), IC8.4 (V+)
- net -15V: now also IC2.11 (V-), IC5.11 (V-), IC8.11 (V-)

Commit message: vcf-24 pcb
Parts:
- C10, C11, C12, C13, C14, C15, C16, C17, C18: footprint FormantKO:C_Rect -> FormantKO:C_Rect_300_400
- J4: value IS_SELECT -> IS SELECT
- J5: value OS_SELECT -> IOS SELECT
Connections:
- net -15V: now also C13.1, C17.1; no longer C13.2, C17.2
- net GND: now also C13.2, C17.2; no longer C13.1, C17.1
- net OS renamed IOS
Other:
- moved on the sheet: C13, C17
Changed lines of the file:
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@@
 		)
 	)
-	(global_label "OS"
+	(global_label "IOS"
 		(shape input)
 		(at 67.31 104.14 180)
@@
 		)
 		(property "Intersheetrefs" "${INTERSHEET_REFS}"
-			(at 61.6897 104.14 0)
+			(at 61.0849 104.14 0)
 			(hide yes)
 			(show_name no)
@@
 	(symbol
 		(lib_id "FormantKO:C")
-		(at 88.9 171.45 0)
+		(at 88.9 171.45 180)
 		(unit 1)
 		(body_style 1)
@@
 					(size 1.27 1.27)
 				)
-				(justify right)
+				(justify left)
 			)
 		)
@@
 					(size 1.27 1.27)
 				)
-				(justify left)
+				(justify right)
 			)
 		)
-		(property "Footprint" "FormantKO:C_Rect"
+		(property "Footprint" "FormantKO:C_Rect_300_400"
 			(at 88.9 171.45 0)
 			(hide yes)
@@
 		(lib_id "FormantKO:C")
 		(at 88.9 158.75 0)
+		(mirror y)
 		(unit 1)
 		(body_style 1)
@@
 					(size 1.27 1.27)
 				)
-				(justify right)
+				(justify left)
 			)
 		)
@@
 					(size 1.27 1.27)
 				)
-				(justify left)
+				(justify right)
 			)
 		)
-		(property "Footprint" "FormantKO:C_Rect"
+		(property "Footprint" "FormantKO:C_Rect_300_400"
 			(at 88.9 158.75 0)
 			(hide yes)
@@
 	(symbol
 		(lib_id "FormantKO:C")
-		(at 63.5 171.45 0)
+		(at 63.5 171.45 180)
 		(unit 1)
 		(body_style 1)
@@
 					(size 1.27 1.27)
 				)
-				(justify right)
+				(justify left)
 			)
 		)
@@
 					(size 1.27 1.27)
 				)
-				(justify left)
+				(justify right)
 			)
 		)
-		(property "Footprint" "FormantKO:C_Rect"
+		(property "Footprint" "FormantKO:C_Rect_300_400"
 			(at 63.5 171.45 0)
 			(hide yes)
@@
 			)
 		)
-		(property "Footprint" "FormantKO:C_Rect"
+		(property "Footprint" "FormantKO:C_Rect_300_400"
 			(at 76.2 158.75 0)
 			(hide yes)
@@
 			)
 		)
-		(property "Footprint" "FormantKO:C_Rect"
+		(property "Footprint" "FormantKO:C_Rect_300_400"
 			(at 63.5 158.75 0)
 			(hide yes)
@@
 			)
 		)
-		(property "Value" "OS_SELECT"
+		(property "Value" "IOS SELECT"
 			(at 76.2 99.06 0)
 			(show_name no)
@@
 			)
 		)
-		(property "Footprint" "FormantKO:C_Rect"
+		(property "Footprint" "FormantKO:C_Rect_300_400"
 			(at 50.8 171.45 0)
 			(hide yes)
@@
 			)
 		)
-		(property "Value" "IS_SELECT"
+		(property "Value" "IS SELECT"
 			(at 76.2 66.04 0)
 			(show_name no)
@@
 			)
 		)
-		(property "Footprint" "FormantKO:C_Rect"
+		(property "Footprint" "FormantKO:C_Rect_300_400"
 			(at 101.6 171.45 0)
 			(hide yes)
@@
 			)
 		)
-		(property "Footprint" "FormantKO:C_Rect"
+		(property "Footprint" "FormantKO:C_Rect_300_400"
 			(at 76.2 171.45 0)
 			(hide yes)
@@
 			)
 		)
-		(property "Footprint" "FormantKO:C_Rect"
+		(property "Footprint" "FormantKO:C_Rect_300_400"
 			(at 50.8 158.75 0)
 			(hide yes)
