File: modules/VCF_24/system.kicad_sch (KiCad schematic)
At the start: 23 parts, among them IC2 TL074, IC5 TL074, IC8 TL074, J1 BUS CONNECTOR, J2 KOV SELECT, J3 ENV SELECT, J4 IS SELECT, J5 IOS SELECT, J6 ECV, J7 TM, J8 ES, J9 EOS

Commit message: vcf-24 pcb
Connections:
- net +15V: now also C10.2; no longer C10.1
- net -15V: now also C11.1; no longer C11.2
- net GND: now also C10.1, C11.2; no longer C10.2, C11.1
Other:
- moved on the sheet: C10, C11
Changed lines of the file:
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@@
 	(symbol
 		(lib_id "FormantKO:C")
-		(at 50.8 171.45 0)
+		(at 50.8 171.45 180)
 		(unit 1)
 		(body_style 1)
@@
 					(size 1.27 1.27)
 				)
+				(justify left)
+			)
+		)
+		(property "Value" "100n"
+			(at 52.07 175.26 0)
+			(show_name no)
+			(do_not_autoplace no)
+			(effects
+				(font
+					(size 1.27 1.27)
+				)
 				(justify right)
-			)
-		)
-		(property "Value" "100n"
-			(at 52.07 173.99 0)
-			(show_name no)
-			(do_not_autoplace no)
-			(effects
-				(font
-					(size 1.27 1.27)
-				)
-				(justify left)
 			)
 		)
@@
 	(symbol
 		(lib_id "FormantKO:C")
-		(at 50.8 158.75 0)
+		(at 50.8 158.75 180)
 		(unit 1)
 		(body_style 1)
@@
 					(size 1.27 1.27)
 				)
-				(justify right)
+				(justify left)
 			)
 		)
@@
 					(size 1.27 1.27)
 				)
-				(justify left)
-			)
-		)
+				(justify right)
+			)
+		)
