File: modules/VCF_24/vcf_24b.kicad_sch (KiCad schematic)
At the start: 38 parts, among them IC2 TL074, IC3 CA3080, IC4 CA3080, IC8 TL074, P4 100k, P5 47k

Commit message: vcf-24 pcb
Parts:
- removed S2: SW, symbol FormantKO:SW_SPDT_x4
- removed S3: SW, symbol FormantKO:SW_SPDT_x2
- added S2.1, S2.2: MODE, FormantKO:PanelConnector_1x03, symbol FormantKO:SW_SPDT
- added S4.1, S4.2: TOPO, FormantKO:PanelConnector_1x03, symbol FormantKO:SW_SPDT
- C3: footprint FormantKO:C_Rect -> FormantKO:C_Rect_200
- C4, C5: footprint FormantKO:C_Rect -> FormantKO:C_Rect_200; Note (none) -> *
- C9: footprint FormantKO:C_Rect -> FormantKO:C_Rect_300_400
- R49: Note (none) -> *
Connections:
- net GND: now also S4.2.3 (b)
- net IS: now also S4.1.3 (b), S4.2.1 (a)
- net W: now also S2.2.2 (c)
- net X: now also S2.1.2 (c)
- net at IC2.1, R21.2, R22.2: now also S2.2.3 (b)
- net at IC8.1, R54.2: now also S4.1.1 (a)
- net at R51.1: now also S4.1.2 (c)
- net at IC2.14, R15.2, R16.2: now also S2.1.3 (b)
- net at R55.1: now also S4.2.2 (c)
- net at IC2.8, IC2.9 (-), R14.2: now also S2.1.1 (a)
- net at IC2.6 (-), IC2.7, R20.2: now also S2.2.1 (a)
- net A renamed V
Other:
- moved on the sheet: R49
