File: modules/VCF_24/vcf_24c.kicad_sch (KiCad schematic)
At the start: 23 parts, among them IC5 TL074, IC6 CA3080, IC7 CA3080, IC8 TL074

Commit message: vcf-24 pcb
Parts:
- removed S2: SW, symbol FormantKO:SW_SPDT_x4
- added C8: 150p, FormantKO:C_Rect_300_400, symbol FormantKO:C
- added P6: 47k, FormantKO:PanelConnector_1x03, symbol FormantKO:R_Potentiometer
- added R45, R46, R47, R50: 39k, FormantKO:R_Axial_Horizontal, symbol FormantKO:R
- added R48: 470R, FormantKO:R_Axial_Horizontal, symbol FormantKO:R
- added R57: 82k, FormantKO:R_Axial_Horizontal, symbol FormantKO:R
- added S2.3, S2.4: MODE, FormantKO:PanelConnector_1x03, symbol FormantKO:SW_SPDT
- added S3.1, S3.2: POLES, FormantKO:PanelConnector_1x06, symbol FormantKO:SW_SP4T
- C6, C7: footprint FormantKO:C_Rect -> FormantKO:C_Rect_200; Note (none) -> *
Connections:
- net GND: now also P6.1, R57.2, S3.2.1, S3.2.3
- net W: now also S3.1.2
- net X: now also S3.1.1
- net Y: now also S2.4.2 (c), S3.1.4
- net Z: now also R50.1
- net at IC5.6 (-), IC5.7, R32.2: now also S2.4.1 (a)
- net at IC5.1, R33.2, R34.2: now also S2.4.3 (b)
- net at IC5.8, IC5.9 (-), R26.2: now also S2.3.1 (a)
- net at R31.1: now also S2.3.2 (c), S3.1.3
- net at IC5.14, R27.2, R28.2: now also S2.3.3 (b)
- net at IC8.10 (+): now also R46.2, R57.1, S3.2.6 (C)
- net at IC8.8: now also R47.2, R48.1
- net at IC8.9 (-): now also R45.2, R47.1, R50.2
- new net: C8.1, P6.3, R48.2
- new net: R45.1, R46.1, S3.1.6 (C)
- new net EOS: C8.2
- new net IOS: P6.2
- no-connect marks 0 -> 2
Other:
- note removed: "*"
- moved on the sheet: IC8C
