File: modules/VCF_24/vcf_24c.kicad_sch (KiCad schematic)
At the start: 34 parts, among them IC5 TL074, IC6 CA3080, IC7 CA3080, IC8 TL074, P6 47k

Commit message: vcf-24 pcb
Connections:
- net EOS: now also C8.1; no longer C8.2
- net at P6.3, R48.2: now also C8.2; no longer C8.1
Other:
- moved on the sheet: C8
Changed lines of the file:
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@@
 	(symbol
 		(lib_id "FormantKO:C")
-		(at 158.75 124.46 90)
+		(at 158.75 124.46 270)
 		(unit 1)
 		(body_style 1)
@@
 		(dnp no)
 		(property "Reference" "C8"
-			(at 157.734 120.65 90)
+			(at 158.75 120.65 90)
 			(show_name no)
 			(do_not_autoplace no)
@@
 		)
 		(property "Value" "150p"
-			(at 160.782 128.27 90)
+			(at 158.75 128.27 90)
 			(show_name no)
 			(do_not_autoplace no)
