File: modules/KBI/system.kicad_sch (KiCad schematic)
At the start: 16 parts, among them J1 +15V, J10 D, J11 E, J12 F, J13 G, J2 -15V, J3 GND, J4 KOV, J6 FM, J7 A, J8 B, J9 C

Commit message: added card extender to system
Parts:
- added C7, C8, C9: 680n, FormantKO:C_Rect, symbol FormantKO:C
- H1, H2, H3, H4: footprint FormantKO:MountingHole_3.2mm_M3 -> FormantKO:MountingHole_2.7mm_M2.5
Connections:
- net +15V: now also C7.1, C8.1
- net -15V: now also C8.2, C9.2
- net GND: now also C7.2, C9.1
Other:
- moved on the sheet: J6
