File: mixer/modules/CHANNEL/CHANNEL.kicad_pcb (KiCad board)
At the start: 2 copper layers, 160 x 233.3 mm, 3 parts, among them J1 MixerBus

Commit message: com rework; channel first stab at schematic
Parts:
- added C1: 50n, FormantKO:C_Rect, F.Cu at (55.5, 211.9)
- added C10: 100n, FormantKO:C_Rect, F.Cu at (158.4, 183.0)
- added C11: 10µ, FormantKO:CP_Axial_600, F.Cu at (163.3, 170.2)
- added C12: 100n, FormantKO:C_Rect, F.Cu at (96.1, 189.0)
- added C13: 100n, FormantKO:C_Rect, F.Cu at (158.4, 186.8)
- added C2: 5n, FormantKO:C_Rect, F.Cu at (131.7, 194.1)
- added C3: 22n, FormantKO:C_Rect, F.Cu at (146.9, 184.0)
- added C4: 10p, FormantKO:C_Rect, F.Cu at (169.0, 213.0)
- added C5: 5n, FormantKO:C_Rect, F.Cu at (157.1, 191.6)
- added C6: 100n, FormantKO:C_Rect, F.Cu at (139.0, 204.0)
- added C7: 100n, FormantKO:C_Rect, F.Cu at (96.1, 184.0)
- added C8: 10µ, FormantKO:CP_Axial_600, F.Cu at (163.3, 163.8)
- added C9: 100n, FormantKO:C_Rect, F.Cu at (93.6, 194.1)
- added IC1: OpAmp, FormantKO:DIP-8, F.Cu at (80.9, 184.0)
- added IC2: OpAmp, FormantKO:DIP-8, F.Cu at (113.9, 196.7)
- added J1: ES, FormantKO:PanelConnector_1x02, F.Cu at (37.7, 162.4)
- added P1: 100k, FormantKO:PanelConnector_1x03, F.Cu at (37.7, 211.9)
- added P10: 100k, FormantKO:PanelConnector_1x03, F.Cu at (58.0, 237.3)
- added P2: 100k, FormantKO:PanelConnector_1x03, F.Cu at (37.7, 199.2)
- added P3: 100k, FormantKO:PanelConnector_1x03, F.Cu at (37.7, 186.5)
- added P4: 50k, FormantKO:PanelConnector_1x03, F.Cu at (37.7, 224.6)
- added P5: 100k, FormantKO:PanelConnector_1x03, F.Cu at (37.7, 173.8)
- added P6: 100k, FormantKO:PanelConnector_1x03, F.Cu at (37.7, 237.3)
- added P7: 100k, FormantKO:PanelConnector_1x03, F.Cu at (47.9, 224.6)
- added P8: 100k, FormantKO:PanelConnector_1x03, F.Cu at (47.9, 237.3)
- added P9: 100k, FormantKO:PanelConnector_1x03, F.Cu at (58.0, 224.6)
- added R1: 11k, FormantKO:R_Axial_Horizontal, F.Cu at (58.0, 168.7)
- added R10: 120k, FormantKO:R_Axial_Horizontal, F.Cu at (131.7, 178.9)
- added R11: 47k, FormantKO:R_Axial_Horizontal, F.Cu at (153.0, 204.0)
- added R12: 120k, FormantKO:R_Axial_Horizontal, F.Cu at (106.3, 166.2)
- added R13: 120k, FormantKO:R_Axial_Horizontal, F.Cu at (119.0, 222.1)
- added R14: 22k, FormantKO:R_Axial_Horizontal, F.Cu at (168.0, 217.0)
- added R15: 22k, FormantKO:R_Axial_Horizontal, F.Cu at (144.4, 237.3)
- added R16: 22k, FormantKO:R_Axial_Horizontal, F.Cu at (168.0, 222.0)
- added R17: 22k, FormantKO:R_Axial_Horizontal, F.Cu at (144.4, 242.4)
- added R18: 22k, FormantKO:R_Axial_Horizontal, F.Cu at (168.0, 209.0)
- added R19: 22k, FormantKO:R_Axial_Horizontal, F.Cu at (144.4, 232.2)
- added R2: 11k, FormantKO:R_Axial_Horizontal, F.Cu at (70.7, 214.4)
- added R20: 22k, FormantKO:R_Axial_Horizontal, F.Cu at (168.0, 227.0)
- added R21: 22k, FormantKO:R_Axial_Horizontal, F.Cu at (144.4, 225.0)
- added R3: 11k, FormantKO:R_Axial_Horizontal, F.Cu at (141.8, 214.4)
- added R4: 3k6, FormantKO:R_Axial_Horizontal, F.Cu at (68.2, 201.7)
- added R5: 3k6, FormantKO:R_Axial_Horizontal, F.Cu at (124.0, 206.8)
- added R6: 470k, FormantKO:R_Axial_Horizontal, F.Cu at (168.0, 204.0)
- added R7: 1k8, FormantKO:R_Axial_Horizontal, F.Cu at (58.0, 176.3)
- added R8: 1k8, FormantKO:R_Axial_Horizontal, F.Cu at (58.0, 189.0)
- added R9: 120k, FormantKO:R_Axial_Horizontal, F.Cu at (106.3, 161.1)
- renumbered J1 to J2
Connections:
- J2 pad a2: unconnected-(J1-MBL-Pada2) -> MBL
- J2 pad a24: unconnected-(J1-X1L-Pada24) -> X1L
- J2 pad a26: unconnected-(J1-X2L-Pada26) -> X2L
- J2 pad a28: unconnected-(J1-X3L-Pada28) -> X3L
- J2 pad a30: unconnected-(J1-X4L-Pada30) -> X4L
- J2 pad b2: unconnected-(J1-MBR-Padb2) -> MBR
- J2 pad b24: unconnected-(J1-X1R-Padb24) -> X1R
- J2 pad b26: unconnected-(J1-X2R-Padb26) -> X2R
- J2 pad b28: unconnected-(J1-X3R-Padb28) -> X3R
- J2 pad b30: unconnected-(J1-X4R-Padb30) -> X4R
