File: sequencer/modules/CLOCK/CLOCK.kicad_pcb (KiCad board)
At the start: 2 copper layers, 160 x 100 mm, 37 parts, among them J1 Card_Connector, J10 XSTP, J2 XCLK, J3 CKOUT, J4 STUP, J5 STDN, J6 STRN, J7 RST, J8 TRIG, J9 GATE, U1 40106, U2 40106, U3 4013

Commit message: clock work
Parts:
- removed J10: XSTP, FormantKO:PanelConnector_1x02
- removed J9: GATE, FormantKO:PanelConnector_1x02
- removed LED1: DLED, FormantKO:PanelConnector_1x02
- removed S4: STOP/RUN, FormantKO:PanelConnector_1x02
- added C1: 10n, FormantKO:C_Rect_200, F.Cu at (82.9, 129.3)
- added C2: 20n, FormantKO:C_Rect_200, F.Cu at (91.8, 129.3)
- added C3: 10n, FormantKO:C_Rect_200, F.Cu at (104.5, 129.3)
- added C4: 20n, FormantKO:C_Rect_200, F.Cu at (113.4, 129.3)
- added C5: 20n, FormantKO:C_Rect_200, F.Cu at (79.1, 89.9)
- added C6: 20n, FormantKO:C_Rect_200, F.Cu at (112.1, 84.8)
- added C7: 10n, FormantKO:C_Rect_200, F.Cu at (112.1, 79.8)
- added D1: DUS, FormantKO:DUS_300, F.Cu at (93.1, 86.1)
- added D11: DUS, FormantKO:DUS_300, F.Cu at (89.3, 86.1)
- added D2: DUS, FormantKO:DUS_300, F.Cu at (96.9, 86.1)
- added D3: DUS, FormantKO:DUS_300, F.Cu at (91.8, 97.5)
- added D4: DUS, FormantKO:DUS_300, F.Cu at (91.8, 101.3)
- added D5: DUS, FormantKO:DUS_300, F.Cu at (99.4, 98.8)
- added D6: DUS, FormantKO:DUS_300, F.Cu at (102.0, 93.7)
- added D7: DUS, FormantKO:DUS_300, F.Cu at (124.8, 95.0)
- added D8: DUS, FormantKO:DUS_300, F.Cu at (91.8, 105.2)
- added R1: 10k, FormantKO:R_Axial_Horizontal_400, F.Cu at (77.8, 129.3)
- added R10: 10k, FormantKO:R_Axial_Horizontal_400, F.Cu at (107.1, 101.3)
- added R11: 10k, FormantKO:R_Axial_Horizontal_400, F.Cu at (107.1, 105.2)
- added R12: 47k, FormantKO:R_Axial_Horizontal_400, F.Cu at (138.8, 54.4)
- added R13: 1M, FormantKO:R_Axial_Horizontal_400, F.Cu at (79.1, 86.1)
- added R14: 1M, FormantKO:R_Axial_Horizontal_400, F.Cu at (79.1, 95.0)
- added R15: 680k, FormantKO:R_Axial_Horizontal_400, F.Cu at (122.3, 84.8)
- added R16: 220k, FormantKO:R_Axial_Horizontal_400, F.Cu at (112.1, 88.7)
- added R17: 10k, FormantKO:R_Axial_Horizontal_400, F.Cu at (118.5, 79.8)
- added R2: 680k, FormantKO:R_Axial_Horizontal_400, F.Cu at (86.7, 129.3)
- added R3: 220k, FormantKO:R_Axial_Horizontal_400, F.Cu at (95.6, 129.3)
- added R4: 47k, FormantKO:R_Axial_Horizontal_400, F.Cu at (79.1, 82.3)
- added R40: 47k, FormantKO:R_Axial_Horizontal_400, F.Cu at (129.9, 114.0)
- added R5: 10k, FormantKO:R_Axial_Horizontal_400, F.Cu at (99.4, 129.3)
- added R6: 680k, FormantKO:R_Axial_Horizontal_400, F.Cu at (108.3, 129.3)
- added R7: 220k, FormantKO:R_Axial_Horizontal_400, F.Cu at (117.2, 129.3)
- added R8: 47k, FormantKO:R_Axial_Horizontal_400, F.Cu at (79.1, 78.5)
- added R9: 100k, FormantKO:R_Axial_Horizontal_400, F.Cu at (84.2, 120.4)
- added TP1: TestPoint, FormantKO:KEYSTONE_5001, F.Cu at (103.2, 79.8)
- added U4: 40193, FormantKO:DIP-16, F.Cu at (149.0, 65.8)
- C11, C22, C8, C9: footprint FormantKO:C_Rect -> FormantKO:C_Rect_200
- D31, D9: footprint FormantKO:DUS -> FormantKO:DUS_300
- J2: value XCLK -> CKOUT; footprint FormantKO:PanelConnector_1x02 -> FormantKO:Wire_1x01_General
- J3: value CKOUT -> RST; footprint FormantKO:PanelConnector_1x02 -> FormantKO:Wire_1x01_General
- J4: value STUP -> RIN; footprint FormantKO:PanelConnector_1x02 -> FormantKO:Wire_1x01_General
- J5: value STDN -> CLR; footprint FormantKO:PanelConnector_1x02 -> FormantKO:Wire_1x01_General
- J6: value STRN -> RND; footprint FormantKO:PanelConnector_1x02 -> FormantKO:Wire_1x01_General
- J7: value RST -> STUP; footprint FormantKO:PanelConnector_1x02 -> FormantKO:Wire_1x01_General
- J8: value TRIG -> STDN; footprint FormantKO:PanelConnector_1x02 -> FormantKO:Wire_1x01_General
- R18, R20, R21, R22, R23, R24, R41, R42, R43, R44, R45, R46, R47: footprint FormantKO:R_Axial_Horizontal -> FormantKO:R_Axial_Horizontal_400
- moved R47 89.3 mm to (70.2, 124.2)
- moved C11 84.6 mm to (67.7, 133.1)
- moved J6 80.4 mm to (147.7, 54.4), turned to 0 degrees
- moved J7 76.3 mm to (82.9, 138.2), turned to 0 degrees
- moved D31 73.9 mm to (114.7, 54.4)
- moved R20 70.8 mm to (121.0, 129.3), turned to -90 degrees
- moved R21 70.6 mm to (138.8, 129.3), turned to 90 degrees
- moved R22 69.9 mm to (129.9, 129.3), turned to 90 degrees
- moved J2 69.1 mm to (91.8, 53.1), turned to 0 degrees
- moved U3 67.4 mm to (79.1, 107.7), turned to 0 degrees
- moved J3 61.0 mm to (117.2, 62.0), turned to 0 degrees
- moved J4 59.9 mm to (124.8, 62.0), turned to 0 degrees
- moved J5 58.3 mm to (123.6, 54.4), turned to 0 degrees
- moved R44 58.3 mm to (65.2, 97.5), turned to -90 degrees
- moved C22 57.9 mm to (67.7, 107.7)
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Connections:
- J2 pad 1: GND -> CKOUT
- J3 pad 1: GND -> RST
- J4 pad 1: +15V -> RIN
- J5 pad 1: +15V -> CLR
- J6 pad 1: +15V -> RND
- J7 pad 1: GND -> STUP
- J8 pad 1: GND -> STDN
- U1 pad 1: unconnected-(U1-Pad1) -> Net-(C2-Pad2)
- U1 pad 10: unconnected-(U1-Pad10) -> Net-(D6-K)
- U1 pad 11: unconnected-(U1-Pad11) -> Net-(D8-A)
- U1 pad 12: unconnected-(U1-Pad12) -> Net-(D5-K)
- U1 pad 13: unconnected-(U1-Pad13) -> Net-(D4-A)
- U1 pad 2: unconnected-(U1-Pad2) -> Net-(D1-K)
- U1 pad 3: unconnected-(U1-Pad3) -> Net-(C4-Pad2)
- U1 pad 4: unconnected-(U1-Pad4) -> Net-(D2-K)
- U2 pad 1: unconnected-(U2-Pad1) -> Net-(D2-A)
- U2 pad 10: unconnected-(U2-Pad10) -> UP
- U2 pad 11: unconnected-(U2-Pad11) -> Net-(U2-Pad11)
- U2 pad 12: unconnected-(U2-Pad12) -> Net-(U2-Pad11)
- U2 pad 13: unconnected-(U2-Pad13) -> Net-(D1-A)
- U2 pad 2: unconnected-(U2-Pad2) -> Net-(U2-Pad2)
- U2 pad 3: unconnected-(U2-Pad3) -> Net-(U2-Pad2)
- U2 pad 4: unconnected-(U2-Pad4) -> DN
- U2 pad 5: unconnected-(U2-Pad5) -> Net-(C6-Pad2)
- U2 pad 6: unconnected-(U2-Pad6) -> RST
- U3 pad 10: unconnected-(U3B-R-Pad10) -> Net-(U3B-R)
- U3 pad 11: unconnected-(U3B-C-Pad11) -> GND
- U3 pad 12: unconnected-(U3B-~{Q}-Pad12) -> Net-(D8-K)
- U3 pad 13: unconnected-(U3B-Q-Pad13) -> Net-(D4-K)
- U3 pad 8: unconnected-(U3B-S-Pad8) -> Net-(D11-K)
- U3 pad 9: unconnected-(U3B-D-Pad9) -> GND
Other:
- board text added: "${COMMENT1} | MFOS"
- board text added: "| ${COMPANY} MFOS | ${COMMENT1} ${TITLE} | REVISION ${REVISION} | ${ISSUE_DATE} |"
- board text removed: "${COMMENT1}"
- board text removed: "| ${COMPANY} | ${COMMENT1} ${TITLE} | REVISION ${REVISION} | ${ISSUE_DATE} |"

Commit message: sequencer clock work
Parts:
- added C15: 10n, FormantKO:C_Rect_160, F.Cu at (176.9, 117.9)
- added C16: 10n, FormantKO:C_Rect_160, F.Cu at (197.2, 92.5)
- added C17: 100p, FormantKO:C_Rect_160, F.Cu at (143.9, 88.7)
- added C18: 1n, FormantKO:C_Rect_160, F.Cu at (161.7, 82.3)
- added C19: 100n, FormantKO:C_Rect_160, F.Cu at (71.2, 83.8)
- added C20: 10µ, Capacitor_THT:CP_Radial_D5.0mm_P2.50mm, F.Cu at (184.5, 131.9)
- added C21: 10µ, Capacitor_THT:CP_Radial_D5.0mm_P2.50mm, F.Cu at (192.2, 134.4)
- added C24: 100n, FormantKO:C_Rect_160, F.Cu at (142.6, 103.9)
- added D30: DUS, FormantKO:DUS_300, F.Cu at (182.8, 101.3)
- added J10: STRN, FormantKO:Wire_1x01_General, F.Cu at (134.2, 135.6)
- added J11: STP, FormantKO:Wire_1x01_General, F.Cu at (61.8, 117.9)
- added J12: XSTP, FormantKO:Wire_1x01_General, F.Cu at (66.2, 88.9)
- added J13: REV, FormantKO:Wire_1x01_General, F.Cu at (72.3, 74.2)
- added J9: XCLK, FormantKO:Wire_1x01_General, F.Cu at (112.9, 135.6)
- added Q1: 2N3904, Package_TO_SOT_THT:TO-92_Inline_Wide, F.Cu at (194.7, 122.9)
- added R31: 2M, FormantKO:R_Axial_Horizontal_400, F.Cu at (182.0, 122.9)
- added R32: 100k, FormantKO:R_Axial_Horizontal_400, F.Cu at (185.8, 110.2)
- added R33: 1M, FormantKO:R_Axial_Horizontal_400, F.Cu at (193.4, 110.2)
- added R34: 4k7, FormantKO:R_Axial_Horizontal_400, F.Cu at (182.0, 93.7)
- added R35: 2M, FormantKO:R_Axial_Horizontal_400, F.Cu at (197.2, 110.2)
- added R36: 4M7, FormantKO:R_Axial_Horizontal_400, F.Cu at (189.6, 110.2)
- added R37: 4k7, FormantKO:R_Axial_Horizontal_400, F.Cu at (196.0, 96.3)
- added R38: 1M, FormantKO:R_Axial_Horizontal_400, F.Cu at (173.1, 86.1)
- added R39: 10k, FormantKO:R_Axial_Horizontal_400, F.Cu at (149.0, 82.3)
- added U6: 40106, FormantKO:DIP-14, F.Cu at (192.2, 78.5)
- added U7: TL082, FormantKO:DIP-8, F.Cu at (176.7, 110.2)
- added U8: 4514, FormantKO:DIP-24W, F.Cu at (161.9, 95.9)
- C1, C2, C22, C3, C4, C5, C6, C7, C8, C9: footprint FormantKO:C_Rect_200 -> FormantKO:C_Rect_160
- C10: footprint Capacitor_THT:CP_Radial_D5.0mm_P2.50mm -> Capacitor_THT:CP_Radial_Tantal_D5.5mm_P2.50mm
- C23: renamed from C11; footprint FormantKO:C_Rect_200 -> FormantKO:C_Rect_160
- moved TP1 25.4 mm to (88.0, 59.4)
- moved C23 20.3 mm to (68.2, 112.8)
- moved D9 7.89 mm to (127.1, 106.9)
- moved U4 6.35 mm to (149.0, 72.1)
- moved C10 4.58 mm to (119.0, 111.3)
- moved U2 4.32 mm to (98.2, 73.9)
- moved J7 3.59 mm to (80.4, 135.6)
- moved R42 2.90 mm to (144.9, 127.5)
- moved J8 2.84 mm to (103.2, 135.6)
- moved R23 2.84 mm to (119.8, 106.4), turned to 180 degrees
- moved D2 2.75 mm to (94.6, 87.6)
- moved C1 2.70 mm to (80.9, 127.5)
- moved R40 2.18 mm to (131.2, 112.3), turned to -90 degrees
- moved C2 2.18 mm to (90.5, 127.5)
- moved C3 2.18 mm to (103.2, 127.5)
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Routing:
- net GND: track 0.00 -> 180.3 mm
- net Net-(C9-Pad2): track 0.00 -> 46.7 mm
- net Net-(D2-K): track 0.00 -> 35.7 mm
- net Net-(D1-K): track 0.00 -> 31.7 mm
- net Net-(C4-Pad2): track 0.00 -> 30.0 mm
- net REV: track 0.00 -> 29.5 mm
- net Net-(U3B-R): track 0.00 -> 29.0 mm
- net Net-(D1-A): track 0.00 -> 25.8 mm
- net Net-(C1-Pad2): track 0.00 -> 24.9 mm
- net Net-(C3-Pad2): track 0.00 -> 24.4 mm
- net Net-(C8-Pad2): track 0.00 -> 23.9 mm
- net Net-(D8-A): track 0.00 -> 20.2 mm
- net XSTP: track 0.00 -> 19.7 mm
- net Net-(D2-A): track 0.00 -> 15.7 mm
- net STRN: track 0.00 -> 15.7 mm
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Other:
- board text added: "| ${SRCURL} |"

Commit message: sequencer clock pcb work
Parts:
- removed R19: 1M, FormantKO:PanelConnector_1x03
- added C11: 47p, FormantKO:C_Rect_160, F.Cu at (189.1, 53.9)
- added C12: 1n, FormantKO:C_Rect_200, F.Cu at (191.6, 76.7)
- added C13: 1n, FormantKO:C_Rect_200, F.Cu at (178.9, 64.5)
- added C14: 1n, FormantKO:C_Rect_200, F.Cu at (191.6, 81.3)
- added D13: DUS, FormantKO:DUS_300, F.Cu at (198.5, 53.9)
- added D28: DUS, FormantKO:DUS_300, F.Cu at (129.7, 77.5)
- added D29: DUS, FormantKO:DUS_300, F.Cu at (132.2, 77.5)
- added J14: R19-1&2, FormantKO:Wire_1x01_General, F.Cu at (108.3, 90.9)
- added J15: R19-3, FormantKO:Wire_1x01_General, F.Cu at (104.8, 90.9)
- added J16: QA, FormantKO:Wire_1x01_General, F.Cu at (124.6, 85.9)
- added J17: QB, FormantKO:Wire_1x01_General, F.Cu at (128.1, 85.9)
- added J18: QC, FormantKO:Wire_1x01_General, F.Cu at (132.7, 85.9)
- added J19: QD, FormantKO:Wire_1x01_General, F.Cu at (136.3, 85.9)
- added J20: 0, FormantKO:Wire_2x01_General, F.Cu at (139.3, 130.1)
- added J21: 1, FormantKO:Wire_2x01_General, F.Cu at (142.9, 130.1)
- added J22: 2, FormantKO:Wire_2x01_General, F.Cu at (146.4, 130.1)
- added J23: 3, FormantKO:Wire_2x01_General, F.Cu at (150.0, 130.1)
- added J24: 4, FormantKO:Wire_2x01_General, F.Cu at (153.5, 130.1)
- added J25: 5, FormantKO:Wire_2x01_General, F.Cu at (157.1, 130.1)
- added J26: 6, FormantKO:Wire_2x01_General, F.Cu at (160.7, 130.1)
- added J27: 7, FormantKO:Wire_2x01_General, F.Cu at (164.2, 130.1)
- added J28: 8, FormantKO:Wire_2x01_General, F.Cu at (167.8, 130.1)
- added J29: 9, FormantKO:Wire_2x01_General, F.Cu at (171.3, 130.1)
- added J30: 10, FormantKO:Wire_2x01_General, F.Cu at (174.9, 130.1)
- added J31: 11, FormantKO:Wire_2x01_General, F.Cu at (178.4, 130.1)
- added J32: 12, FormantKO:Wire_2x01_General, F.Cu at (182.0, 130.1)
- added J33: 13, FormantKO:Wire_2x01_General, F.Cu at (185.5, 130.1)
- added J34: 14, FormantKO:Wire_2x01_General, F.Cu at (189.1, 130.1)
- added J35: 15, FormantKO:Wire_2x01_General, F.Cu at (192.7, 130.1)
- added J36: GB, FormantKO:Wire_1x01_General, F.Cu at (166.2, 91.4)
- added J37: CBUS, FormantKO:Wire_1x01_General, F.Cu at (194.2, 59.9)
- added J38: TRIG, FormantKO:Wire_1x01_General, F.Cu at (200.3, 65.0)
- added J39: GATE, FormantKO:Wire_1x01_General, F.Cu at (200.3, 69.1)
- added R25: 4K7, FormantKO:R_Axial_Horizontal_400, F.Cu at (155.6, 88.9)
- added R26: 100k, FormantKO:R_Axial_Horizontal_400, F.Cu at (155.6, 85.3)
- added R27: 1k, FormantKO:R_Axial_Horizontal_400, F.Cu at (191.6, 69.1)
- added R28: 100k, FormantKO:R_Axial_Horizontal_400, F.Cu at (171.3, 60.5)
- added R29: 1k, FormantKO:R_Axial_Horizontal_400, F.Cu at (191.6, 65.0)
- added R30: 3k, FormantKO:R_Axial_Horizontal_400, F.Cu at (185.5, 60.0)
- added U8: HEF4094B, FormantKO:DIP-16, F.Cu at (155.3, 67.8)
- C1, C15, C16, C17, C18, C2, C3, C4, C5, C6, C7, C8, C9: footprint FormantKO:C_Rect_160 -> FormantKO:C_Rect_200
- J1: value Card_Connector -> Sequencer Bus Connector; footprint FormantKO:Card_Connector -> FormantKO:BusConnector_Full_Male_Horizontal
- MH1: footprint FormantKO:Card_Bracket -> FormantKO:CardBracket
- moved U4 18.5 mm to (130.9, 67.8)
- moved C21 17.8 mm to (200.8, 118.8)
- moved C20 16.9 mm to (191.1, 116.3)
- moved U6 16.7 mm to (176.4, 72.9)
- moved D30 15.3 mm to (169.8, 93.2)
- moved U5 15.2 mm to (147.7, 101.1)
- moved C15 14.9 mm to (185.5, 105.7)
- moved R31 14.1 mm to (190.6, 111.8), turned to 180 degrees
- moved TP1 13.0 mm to (75.3, 56.9)
- moved C24 12.8 mm to (130.2, 101.1)
- moved R18 12.3 mm to (110.9, 94.5)
- moved D7 12.2 mm to (113.7, 87.9)
- moved Q1 11.7 mm to (198.2, 111.8), turned to 0 degrees
- moved J5 11.7 mm to (112.4, 57.9)
- moved J4 11.5 mm to (113.4, 62.5)
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- renumbered U8 to U5
Connections:
- D7 pad 2: RST -> Net-(D7-A)
- J1 pad a18: unconnected-(J1-+5V-Pada18) -> +5V
- J1 pad b18: unconnected-(J1-+5V-Padb18) -> +5V
- R17 pad 1: Net-(R17-Pad1) -> RST
- R18 pad 2: Net-(R18-Pad2) -> R19-1&2
- TP1 pad 1: RST -> Net-(D7-A)
- U2 pad 6: RST -> Net-(D7-A)
- U5 pad 10: unconnected-(U8-Q2-Pad10) -> S-2
- U5 pad 11: unconnected-(U8-Q0-Pad11) -> FWD
- U5 pad 13: unconnected-(U8-Q13-Pad13) -> S-13
- U5 pad 14: unconnected-(U8-Q12-Pad14) -> S-12
- U5 pad 15: unconnected-(U8-Q15-Pad15) -> S-15
- U5 pad 16: unconnected-(U8-Q14-Pad16) -> S-14
- U5 pad 17: unconnected-(U8-Q9-Pad17) -> S-9
- U5 pad 18: unconnected-(U8-Q8-Pad18) -> S-8
- U5 pad 19: unconnected-(U8-Q11-Pad19) -> S-11
- U5 pad 20: unconnected-(U8-Q10-Pad20) -> S-10
- U5 pad 4: unconnected-(U8-Q7-Pad4) -> S-7
- U5 pad 5: unconnected-(U8-Q6-Pad5) -> S-6
- U5 pad 6: unconnected-(U8-Q5-Pad6) -> S-5
- U5 pad 7: unconnected-(U8-Q4-Pad7) -> S-4
- U5 pad 8: unconnected-(U8-Q3-Pad8) -> S-3
- U5 pad 9: unconnected-(U8-Q1-Pad9) -> S-1
- U6 pad 10: unconnected-(U6-Pad10) -> Net-(R29-Pad1)
- U6 pad 11: unconnected-(U6-Pad11) -> Net-(C13-Pad2)
- U6 pad 5: unconnected-(U6-Pad5) -> Net-(D28-A)
- U6 pad 6: unconnected-(U6-Pad6) -> Net-(C13-Pad1)
- U6 pad 8: unconnected-(U6-Pad8) -> Net-(R27-Pad1)
- U6 pad 9: unconnected-(U6-Pad9) -> Net-(C13-Pad1)
- U7 pad 4: GND -> -15V
Routing:
- net FWD: track 0.00 -> 228.5 mm, vias 0 -> 2
- net GND: track 180.3 -> 342.6 mm
- net CLK: track 7.11 -> 147.8 mm
- net Net-(U3A-Q): track 0.00 -> 116.2 mm
- net +15V: track 3.56 -> 108.8 mm
- net Net-(D28-A): track 0.00 -> 100.3 mm, vias 0 -> 2
- net CLR: track 0.00 -> 74.8 mm
- net QA: track 0.00 -> 72.2 mm, vias 0 -> 1
- net S-10: track 0.00 -> 69.7 mm, vias 0 -> 2
- net S-14: track 0.00 -> 69.3 mm, vias 0 -> 2
- net S-11: track 0.00 -> 67.5 mm, vias 0 -> 2
- net S-15: track 0.00 -> 67.4 mm, vias 0 -> 2
- net -15V: track 0.00 -> 60.8 mm
- net S-8: track 0.00 -> 55.1 mm
- net S-9: track 0.00 -> 53.8 mm
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