File: sequencer/modules/CLOCK/CLOCK.kicad_sch (KiCad schematic)
At the start: 26 parts, among them U1 40106, U2 40106, U3 4013

Commit message: clock work
Parts:
- C11, C22, C8, C9: footprint FormantKO:C_Rect -> FormantKO:C_Rect_200
- D31, D9: footprint FormantKO:DUS -> FormantKO:DUS_300
- R18, R20, R21, R22, R23, R24, R41, R42, R43, R44, R45, R46, R47: footprint FormantKO:R_Axial_Horizontal -> FormantKO:R_Axial_Horizontal_400
Changed lines of the file:
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@@
 			)
 		)
-		(property "Footprint" "FormantKO:C_Rect"
+		(property "Footprint" "FormantKO:C_Rect_200"
 			(at 139.7 50.8 0)
 			(hide yes)
@@
 			)
 		)
-		(property "Footprint" "FormantKO:DUS"
+		(property "Footprint" "FormantKO:DUS_300"
 			(at 146.05 97.79 0)
 			(hide yes)
@@
 			)
 		)
-		(property "Footprint" "FormantKO:R_Axial_Horizontal"
+		(property "Footprint" "FormantKO:R_Axial_Horizontal_400"
 			(at 146.05 63.5 0)
 			(hide yes)
@@
 			)
 		)
-		(property "Footprint" "FormantKO:R_Axial_Horizontal"
+		(property "Footprint" "FormantKO:R_Axial_Horizontal_400"
 			(at 158.75 104.14 0)
 			(hide yes)
@@
 			)
 		)
-		(property "Footprint" "FormantKO:R_Axial_Horizontal"
+		(property "Footprint" "FormantKO:R_Axial_Horizontal_400"
 			(at 97.79 139.7 0)
 			(hide yes)
@@
 			)
 		)
-		(property "Footprint" "FormantKO:R_Axial_Horizontal"
+		(property "Footprint" "FormantKO:R_Axial_Horizontal_400"
 			(at 71.12 106.68 0)
 			(hide yes)
@@
 			)
 		)
-		(property "Footprint" "FormantKO:R_Axial_Horizontal"
+		(property "Footprint" "FormantKO:R_Axial_Horizontal_400"
 			(at 135.89 104.14 0)
 			(hide yes)
@@
 			)
 		)
-		(property "Footprint" "FormantKO:R_Axial_Horizontal"
+		(property "Footprint" "FormantKO:R_Axial_Horizontal_400"
 			(at 133.35 63.5 0)
 			(hide yes)
@@
 			)
 		)
-		(property "Footprint" "FormantKO:R_Axial_Horizontal"
+		(property "Footprint" "FormantKO:R_Axial_Horizontal_400"
 			(at 222.25 102.87 0)
 			(hide yes)
@@
 			)
 		)
-		(property "Footprint" "FormantKO:C_Rect"
+		(property "Footprint" "FormantKO:C_Rect_200"
 			(at 58.42 106.68 0)
 			(hide yes)
@@
 			)
 		)
-		(property "Footprint" "FormantKO:R_Axial_Horizontal"
+		(property "Footprint" "FormantKO:R_Axial_Horizontal_400"
 			(at 110.49 139.7 0)
 			(hide yes)
@@
 		(exclude_from_sim no)
 		(in_bom yes)
-		(on_board yes)
+		(on_board no)
 		(in_pos_files yes)
 		(dnp no)
@@
 			)
 		)
-		(property "Footprint" "FormantKO:R_Axial_Horizontal"
+		(property "Footprint" "FormantKO:R_Axial_Horizontal_400"
 			(at 135.89 91.44 0)
 			(hide yes)
@@
 			)
 		)
-		(property "Footprint" "FormantKO:DUS"
+		(property "Footprint" "FormantKO:DUS_300"
 			(at 125.73 139.7 0)
 			(hide yes)
@@
 			)
 		)
-		(property "Footprint" "FormantKO:C_Rect"
+		(property "Footprint" "FormantKO:C_Rect_200"
 			(at 104.14 127 0)
 			(hide yes)
@@
 			)
 		)
-		(property "Footprint" "FormantKO:C_Rect"
+		(property "Footprint" "FormantKO:C_Rect_200"
 			(at 77.47 100.33 0)
 			(hide yes)
@@
 			)
 		)
-		(property "Footprint" "FormantKO:R_Axial_Horizontal"
+		(property "Footprint" "FormantKO:R_Axial_Horizontal_400"
 			(at 83.82 106.68 0)
 			(hide yes)
@@
 			)
 		)
-		(property "Footprint" "FormantKO:R_Axial_Horizontal"
+		(property "Footprint" "FormantKO:R_Axial_Horizontal_400"
 			(at 166.37 97.79 0)
 			(hide yes)
@@
 			)
 		)
-		(property "Footprint" "FormantKO:R_Axial_Horizontal"
+		(property "Footprint" "FormantKO:R_Axial_Horizontal_400"
 			(at 58.42 93.98 0)
 			(hide yes)
@@
 			)
 		)
-		(property "Footprint" "FormantKO:R_Axial_Horizontal"
+		(property "Footprint" "FormantKO:R_Axial_Horizontal_400"
 			(at 209.55 110.49 0)
 			(hide yes)
@@
 		(exclude_from_sim no)
 		(in_bom yes)
-		(on_board yes)
+		(on_board no)
 		(in_pos_files yes)
 		(dnp no)
@@
 	(sheet_instances
 		(path "/"
-			(page "1")
-		)
-	)
-	(embedded_fonts no)
+			(page "2")
+		)
+	)
 )

Commit message: sequencer clock work
Parts:
- C10: footprint Capacitor_THT:CP_Radial_D5.0mm_P2.50mm -> Capacitor_THT:CP_Radial_Tantal_D5.5mm_P2.50mm
- C22, C8, C9: footprint FormantKO:C_Rect_200 -> FormantKO:C_Rect_160
- C23: renamed from C11; footprint FormantKO:C_Rect_200 -> FormantKO:C_Rect_160
Changed lines of the file:
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@@
 		(in_pos_files yes)
 		(dnp no)
-		(property "Reference" "C11"
+		(property "Reference" "C23"
 			(at 139.7 46.99 90)
 			(show_name no)
@@
 			)
 		)
-		(property "Footprint" "FormantKO:C_Rect_200"
+		(property "Footprint" "FormantKO:C_Rect_160"
 			(at 139.7 50.8 0)
 			(hide yes)
@@
 			(project "CLOCK"
 				(path "/e63e39d7-6ac0-4ffd-8aa3-1841a4541b55"
-					(reference "C11")
+					(reference "C23")
 					(unit 1)
 				)
@@
 			)
 		)
-		(property "Footprint" "FormantKO:C_Rect_200"
+		(property "Footprint" "FormantKO:C_Rect_160"
 			(at 58.42 106.68 0)
 			(hide yes)
@@
 			)
 		)
-		(property "Footprint" "FormantKO:C_Rect_200"
+		(property "Footprint" "FormantKO:C_Rect_160"
 			(at 104.14 127 0)
 			(hide yes)
@@
 			)
 		)
-		(property "Footprint" "FormantKO:C_Rect_200"
+		(property "Footprint" "FormantKO:C_Rect_160"
 			(at 77.47 100.33 0)
 			(hide yes)
@@
 			)
 		)
-		(property "Footprint" "Capacitor_THT:CP_Radial_D5.0mm_P2.50mm"
+		(property "Footprint" "Capacitor_THT:CP_Radial_Tantal_D5.5mm_P2.50mm"
 			(at 159.7152 120.65 0)
 			(hide yes)
@@
 		)
 		(property "Voltage" "25V"
-			(at 155.448 118.872 0)
+			(at 156.21 118.872 0)
 			(show_name no)
 			(do_not_autoplace no)
@@
 		)
 	)
+	(embedded_fonts no)
 )

Commit message: sequencer clock pcb work
Parts:
- C8, C9: footprint FormantKO:C_Rect_160 -> FormantKO:C_Rect_200
Connections:
- net R19-1&2: now reaches R18.2, R19.2, R19.3
Changed lines of the file:
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@@
 	)
 	(junction
+		(at 172.72 95.25)
+		(diameter 0)
+		(color 0 0 0 0)
+	)
+	(junction
 		(at 204.47 110.49)
 		(diameter 0)
@@
 	)
 	(junction
+		(at 181.61 97.79)
+		(diameter 0)
+		(color 0 0 0 0)
+	)
+	(junction
 		(at 58.42 85.09)
 		(diameter 0)
@@
 	(wire
 		(pts
+			(xy 172.72 90.17) (xy 172.72 95.25)
+		)
+		(stroke
+			(width 0)
+			(type default)
+		)
+	)
+	(wire
+		(pts
 			(xy 104.14 139.7) (xy 106.68 139.7)
 		)
@@
 	(wire
 		(pts
+			(xy 181.61 90.17) (xy 181.61 97.79)
+		)
+		(stroke
+			(width 0)
+			(type default)
+		)
+	)
+	(wire
+		(pts
 			(xy 158.75 107.95) (xy 158.75 110.49)
 		)
@@
 		)
 	)
+	(global_label "R19-3"
+		(shape passive)
+		(at 181.61 90.17 90)
+		(fields_autoplaced yes)
+		(effects
+			(font
+				(size 1.27 1.27)
+			)
+			(justify left)
+		)
+		(property "Intersheetrefs" "${INTERSHEET_REFS}"
+			(at 181.61 81.6348 90)
+			(hide yes)
+			(show_name no)
+			(do_not_autoplace no)
+			(effects
+				(font
+					(size 1.27 1.27)
+				)
+				(justify left)
+			)
+		)
+	)
 	(global_label "CLR"
 		(shape passive)
@@
 		)
 	)
+	(global_label "R19-1&2"
+		(shape passive)
+		(at 172.72 90.17 90)
+		(fields_autoplaced yes)
+		(effects
+			(font
+				(size 1.27 1.27)
+			)
+			(justify left)
+		)
+		(property "Intersheetrefs" "${INTERSHEET_REFS}"
+			(at 172.72 78.8529 90)
+			(hide yes)
+			(show_name no)
+			(do_not_autoplace no)
+			(effects
+				(font
+					(size 1.27 1.27)
+				)
+				(justify left)
+			)
+		)
+	)
 	(global_label "XCLK"
 		(shape passive)
@@
 			)
 		)
-		(property "Footprint" "FormantKO:C_Rect_160"
+		(property "Footprint" "FormantKO:C_Rect_200"
 			(at 58.42 106.68 0)
 			(hide yes)
@@
 		(exclude_from_sim no)
 		(in_bom yes)
-		(on_board yes)
+		(on_board no)
 		(in_pos_files yes)
 		(dnp no)
@@
 			)
 		)
-		(property "Footprint" "FormantKO:C_Rect_160"
+		(property "Footprint" "FormantKO:C_Rect_200"
 			(at 77.47 100.33 0)
 			(hide yes)
