File: sequencer/modules/CLOCK/clock_3.kicad_sch (KiCad schematic)
At the start: 0 parts

Commit message: sequencer clock work
Parts:
- added C15, C16: 10n, FormantKO:C_Rect_160, symbol FormantKO:C
- added C17: 100p, FormantKO:C_Rect_160, symbol FormantKO:C
- added C18: 1n, FormantKO:C_Rect_160, symbol FormantKO:C
- added D30: DUS, FormantKO:DUS_300, symbol FormantKO:DUS
- added Q1: 2N3904, Package_TO_SOT_THT:TO-92_Inline_Wide, symbol Transistor_BJT:2N3904
- added R31, R35: 2M, FormantKO:R_Axial_Horizontal_400, symbol FormantKO:R
- added R32: 100k, FormantKO:R_Axial_Horizontal_400, symbol FormantKO:R
- added R33, R38: 1M, FormantKO:R_Axial_Horizontal_400, symbol FormantKO:R
- added R34, R37: 4k7, FormantKO:R_Axial_Horizontal_400, symbol FormantKO:R
- added R36: 4M7, FormantKO:R_Axial_Horizontal_400, symbol FormantKO:R
- added R39: 10k, FormantKO:R_Axial_Horizontal_400, symbol FormantKO:R
- added U5: HEF4094B, symbol 4xxx:HEF4094B
- added U6: 40106, FormantKO:DIP-14, symbol 4xxx:40106
- added U7: TL082, FormantKO:DIP-8, symbol 4ms_IC:TL082
- added U8: 4514, FormantKO:DIP-24W, symbol 4xxx_IEEE:4514
Connections:
- new net: C15.1, Q1.1 (E), R31.1
- new net: R36.1, R37.2, U7.2 (-)
- new net: R32.1, R33.1, R36.2, U7.1
- new net: D30.1 (K), R34.2, U6.1
- new net: C15.2, R35.2, U7.3 (+)
- new net: C16.2, R33.2, U7.6 (-)
- new net: C17.2, R39.2, U5.1 (STR)
- new net: U5.2 (D), U6.2
- new net: R38.2, U5.3 (CP), U6.4
- new net: C18.2, R38.1, U6.3
- new net: R32.2, U7.5 (+)
- new net: C17.1, U6.12
- new net: D30.2 (A), U7.7
- new net +15V: R31.2, U5.15 (OE), U5.16 (V_{DD}), U8.1 (EL), U8.24 (Vdd)
- new net -15V: Q1.2 (B)
- new net CLK: U6.13
- new net DA: U5.4 (QP0)
- new net DB: U5.5 (QP1)
- new net DC: U5.6 (QP2)
- new net DD: U5.7 (QP3)
- new net GND: C16.1, C18.1, R34.1, R35.1, R37.1, R39.1, U5.8 (V_{SS}), U8.12 (Vss), U8.23 (~{EN})
- new net QA: U8.2 (A0)
- new net QB: U8.3 (A1)
- new net QC: U8.21 (A2)
- new net QD: U8.22 (A3)
- no-connect marks 0 -> 13

Commit message: sequencer clock pcb work
Parts:
- added C11: 47p, FormantKO:C_Rect_160, symbol FormantKO:C
- added C12, C13, C14: 1n, FormantKO:C_Rect_200, symbol FormantKO:C
- added D13, D28, D29: DUS, FormantKO:DUS_300, symbol FormantKO:DUS
- added R25: 4K7, FormantKO:R_Axial_Horizontal_400, symbol FormantKO:R
- added R26, R28: 100k, FormantKO:R_Axial_Horizontal_400, symbol FormantKO:R
- added R27, R29: 1k, FormantKO:R_Axial_Horizontal_400, symbol FormantKO:R
- added R30: 3k, FormantKO:R_Axial_Horizontal_400, symbol FormantKO:R
- C15, C16, C17, C18: footprint FormantKO:C_Rect_160 -> FormantKO:C_Rect_200
- U8: renamed from U5; footprint (none) -> FormantKO:DIP-16
- renumbered U8 to U5
Connections:
- net +15V: now also R28.1
- net GND: now also C12.1, C14.1, R25.1, R30.1
- net at U6.5: now also D28.2 (A), D29.2 (A), R26.2
- net at U6.6: now also U6.9, C13.1
- net at U6.8: now also R27.1
- net at U6.10: now also R29.1
- net at U6.11: now also C13.2, R28.2
- net S-2: now reaches U5.10 (Q2)
- net FWD: now reaches U5.11 (Q0)
- net S-13: now reaches U5.13 (Q13)
- net S-12: now reaches U5.14 (Q12)
- net S-15: now reaches U5.15 (Q15)
- net S-14: now reaches U5.16 (Q14)
- net S-9: now reaches U5.17 (Q9)
- net S-8: now reaches U5.18 (Q8)
- net S-11: now reaches U5.19 (Q11)
- net S-10: now reaches U5.20 (Q10)
- net S-7: now reaches U5.4 (Q7)
- net S-6: now reaches U5.5 (Q6)
- net S-5: now reaches U5.6 (Q5)
- net S-4: now reaches U5.7 (Q4)
- net S-3: now reaches U5.8 (Q3)
- net S-1: now reaches U5.9 (Q1)
- new net CBUS: R30.2
- new net DN: D28.1 (K)
- new net GATE: C12.2, R27.2
- new net GB: R25.2, R26.1
- new net TRIG: C14.2, R29.2
- new net UP: D29.1 (K)
- no-connect marks 13 -> 11
Other:
- moved on the sheet: U5, U6C, U6D, U6E
