File: sequencer/panels/GATE/GATE.kicad_pcb (KiCad board)
At the start: 2 copper layers, 70.8 x 261.8 mm, 5 parts

Commit message: update gate-16 sequencer panel
Parts:
- added REF**: Jack_3.5mm, FormantKO-Panel:Jack_3.5mm, F.Cu at (201.6, 262.2)
- added REF**: Switch_Mini_Toggle, FormantKO-Panel:Switch_Mini_Toggle, F.Cu at (184.6, 171.2)
- added REF**: Jack_3.5mm, FormantKO-Panel:Jack_3.5mm, F.Cu at (176.6, 45.2)
- added REF**: Switch_Mini_Toggle, FormantKO-Panel:Switch_Mini_Toggle, F.Cu at (218.6, 59.2)
- added REF**: Switch_Mini_Toggle, FormantKO-Panel:Switch_Mini_Toggle, F.Cu at (218.6, 143.2)
- added REF**: LED_3mm_6mm_Bezel, FormantKO-Panel:LED_3mm_6mm_Bezel, F.Cu at (192.6, 213.2)
- added REF**: Switch_Mini_Toggle, FormantKO-Panel:Switch_Mini_Toggle, F.Cu at (184.6, 255.2)
- added REF**: Switch_Mini_Toggle, FormantKO-Panel:Switch_Mini_Toggle, F.Cu at (184.6, 115.2)
- added REF**: Jack_3.5mm, FormantKO-Panel:Jack_3.5mm, F.Cu at (176.6, 129.2)
- added REF**: LED_3mm_6mm_Bezel, FormantKO-Panel:LED_3mm_6mm_Bezel, F.Cu at (226.6, 129.2)
- added REF**: Jack_3.5mm, FormantKO-Panel:Jack_3.5mm, F.Cu at (210.6, 185.2)
- added REF**: Jack_3.5mm, FormantKO-Panel:Jack_3.5mm, F.Cu at (210.6, 73.2)
- added REF**: LED_3mm_6mm_Bezel, FormantKO-Panel:LED_3mm_6mm_Bezel, F.Cu at (192.6, 185.2)
- added REF**: Jack_3.5mm, FormantKO-Panel:Jack_3.5mm, F.Cu at (210.6, 45.2)
- added REF**: Jack_3.5mm, FormantKO-Panel:Jack_3.5mm, F.Cu at (210.6, 129.2)
- added REF**: LED_3mm_6mm_Bezel, FormantKO-Panel:LED_3mm_6mm_Bezel, F.Cu at (192.6, 157.2)
- added REF**: Jack_3.5mm, FormantKO-Panel:Jack_3.5mm, F.Cu at (176.6, 101.2)
- added REF**: Switch_Mini_Toggle, FormantKO-Panel:Switch_Mini_Toggle, F.Cu at (184.6, 199.2)
- added REF**: Switch_Mini_Toggle, FormantKO-Panel:Switch_Mini_Toggle, F.Cu at (184.6, 87.2)
- added REF**: Switch_Mini_Toggle, FormantKO-Panel:Switch_Mini_Toggle, F.Cu at (218.6, 87.2)
- added REF**: LED_3mm_6mm_Bezel, FormantKO-Panel:LED_3mm_6mm_Bezel, F.Cu at (192.6, 129.2)
- added REF**: Switch_Mini_Toggle, FormantKO-Panel:Switch_Mini_Toggle, F.Cu at (184.6, 59.2)
- added REF**: LED_3mm_6mm_Bezel, FormantKO-Panel:LED_3mm_6mm_Bezel, F.Cu at (226.6, 185.2)
- added REF**: LED_3mm_6mm_Bezel, FormantKO-Panel:LED_3mm_6mm_Bezel, F.Cu at (192.6, 73.2)
- added REF**: Jack_3.5mm, FormantKO-Panel:Jack_3.5mm, F.Cu at (176.6, 157.2)
- added REF**: Switch_Mini_Toggle, FormantKO-Panel:Switch_Mini_Toggle, F.Cu at (218.6, 199.2)
- added REF**: Switch_Mini_Toggle, FormantKO-Panel:Switch_Mini_Toggle, F.Cu at (184.6, 143.2)
- added REF**: LED_3mm_6mm_Bezel, FormantKO-Panel:LED_3mm_6mm_Bezel, F.Cu at (192.6, 45.2)
- added REF**: Jack_3.5mm, FormantKO-Panel:Jack_3.5mm, F.Cu at (176.6, 241.2)
- added REF**: Jack_3.5mm, FormantKO-Panel:Jack_3.5mm, F.Cu at (210.6, 213.2)
- added REF**: LED_3mm_6mm_Bezel, FormantKO-Panel:LED_3mm_6mm_Bezel, F.Cu at (226.6, 157.2)
- added REF**: Jack_3.5mm, FormantKO-Panel:Jack_3.5mm, F.Cu at (210.6, 241.2)
- added REF**: LED_3mm_6mm_Bezel, FormantKO-Panel:LED_3mm_6mm_Bezel, F.Cu at (226.6, 213.2)
- added REF**: Switch_Mini_Toggle, FormantKO-Panel:Switch_Mini_Toggle, F.Cu at (218.6, 171.2)
- added REF**: LED_3mm_6mm_Bezel, FormantKO-Panel:LED_3mm_6mm_Bezel, F.Cu at (192.6, 241.2)
- added REF**: Switch_Mini_Toggle, FormantKO-Panel:Switch_Mini_Toggle, F.Cu at (184.6, 227.2)
- added REF**: Switch_Mini_Toggle, FormantKO-Panel:Switch_Mini_Toggle, F.Cu at (218.6, 115.2)
- added REF**: Switch_Mini_Toggle, FormantKO-Panel:Switch_Mini_Toggle, F.Cu at (218.6, 227.2)
- added REF**: Jack_3.5mm, FormantKO-Panel:Jack_3.5mm, F.Cu at (176.6, 185.2)
- added REF**: Jack_3.5mm, FormantKO-Panel:Jack_3.5mm, F.Cu at (210.6, 157.2)
- added REF**: Switch_Mini_Toggle, FormantKO-Panel:Switch_Mini_Toggle, F.Cu at (218.6, 255.2)
- added REF**: Jack_3.5mm, FormantKO-Panel:Jack_3.5mm, F.Cu at (176.6, 73.2)
- added REF**: LED_3mm_6mm_Bezel, FormantKO-Panel:LED_3mm_6mm_Bezel, F.Cu at (226.6, 45.2)
- added REF**: LED_3mm_6mm_Bezel, FormantKO-Panel:LED_3mm_6mm_Bezel, F.Cu at (226.6, 101.2)
- added REF**: Jack_3.5mm, FormantKO-Panel:Jack_3.5mm, F.Cu at (210.6, 101.2)
- added REF**: LED_3mm_6mm_Bezel, FormantKO-Panel:LED_3mm_6mm_Bezel, F.Cu at (226.6, 241.2)
- added REF**: LED_3mm_6mm_Bezel, FormantKO-Panel:LED_3mm_6mm_Bezel, F.Cu at (192.6, 101.2)
- added REF**: Jack_3.5mm, FormantKO-Panel:Jack_3.5mm, F.Cu at (176.6, 213.2)
- added REF**: LED_3mm_6mm_Bezel, FormantKO-Panel:LED_3mm_6mm_Bezel, F.Cu at (226.6, 73.2)
Other:
- board text added: "10"
- board text added: "11"
- board text added: "12"
- board text added: "13"
- board text added: "14"
- board text added: "15"
- board text added: "16"
- board text added: "2"
- board text added: "3"
- board text added: "4"
- board text added: "5"
- board text added: "6"
- board text added: "7"
- board text added: "8"
- board text added: "9"
- board text added: "GATE"
- board text removed: "CV"
