File: panels/ADSR/ADSR.kicad_sch (KiCad schematic)
At the start: 4 parts

Commit message: updated ADSR panel to add gate input and change led
Other:
- company: (none) -> THE HOUSE OF GALAHAD
- title: (none) -> ADSR
Changed lines of the file:
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@@
 	(generator "eeschema")
 	(generator_version "10.0")
-	(paper "A4")
+	(paper "USLetter")
+	(title_block
+		(title "ADSR")
+		(date "2026-07-13")
+		(rev "A")
+		(company "THE HOUSE OF GALAHAD")
+		(comment 1 "FORMANT^{KO}")
+	)
 	(symbol
 		(lib_id "FormantKO:Mounting_Hole")
