File: sequencer/modules/GATE/GATE.kicad_pcb (KiCad board)
At the start: 2 copper layers, 160 x 100 mm, 2 parts, among them J1 Card_Connector

Commit message: adsr additions
Parts:
- added U5: 4514, FormantKO:DIP-24W, F.Cu at (135.0, 95.0)
- J1: value Card_Connector -> Sequencer Bus Connector; footprint FormantKO:Card_Connector -> FormantKO:BusConnector_Full_Male_Horizontal
- MH1: footprint FormantKO:Card_Bracket -> FormantKO:CardBracket
Connections:
- J1 pad a18: unconnected-(J1-+5V-Pada18) -> +5V
- J1 pad a4: unconnected-(J1-GATE1-Pada4) -> GATE1
- J1 pad b18: unconnected-(J1-+5V-Padb18) -> +5V
- J1 pad b4: unconnected-(J1-GATE2-Padb4) -> GATE2
