File: modules/VC_LFOs/system.kicad_sch (KiCad schematic)
At the start: 2 parts, among them J1 Card_Connector

Commit message: vc-lfo schematic; pcb start
Parts:
- added C3, C4: 100µ, FormantKO:CP_Axial_600, symbol FormantKO:C_Polarized
- added IC2, IC4: LM324, FormantKO:DIP-14, symbol FormantKO:LM324
- added J2, J3, J4, J5, J6, J7, J8, J9: MonoJack, FormantKO:PanelConnector_1x02, symbol FormantKO:MonoJack
- J1: footprint FormantKO:Card_Connector -> FormantKO:CardConnector; symbol FormantKO:Card_Connector -> FormantKO:CardConnector
- MH1: value (none) -> CardBracket; footprint FormantKO:Schroff_60807-011_3U_Pair -> FormantKO:CardBracket; symbol FormantKO:Card_Bracket -> FormantKO:CardBracket
Connections:
- net +15V: now also C3.1, IC2.4 (V+), IC4.4 (V+)
- net -15V: now also C4.2, IC2.11 (V-), IC4.11 (V-)
- net GND: now also C3.2, C4.1, J2.1 (S), J3.1 (S), J4.1 (S), J5.1 (S), J6.1 (S), J7.1 (S), J8.1 (S), J9.1 (S)
- new net A: J2.2 (T), J3.2 (T)
- new net RAMP1: J4.2 (T)
- new net RAMP2: J8.2 (T)
- new net SAW2: J7.2 (T)
- new net SQUARE1: J5.2 (T)
- new net TRIANGLE1: J6.2 (T)
- new net TRIANGLE2: J9.2 (T)

Commit message: vc-lfos pcb and schematic fix for opamp orientations
Parts:
- added IC5: LM324, FormantKO:DIP-14, symbol FormantKO:LM324
- J2: Legend LEGEND -> ECVA
- J3: Legend LEGEND -> ECVB
- J4: Legend LEGEND -> RAMP1
- J5: Legend LEGEND -> SQUARE1
- J6: Legend LEGEND -> TRIANGLE1
- J7: Legend LEGEND -> SAW2
- J8: Legend LEGEND -> RAMP2
- J9: Legend LEGEND -> TRIANGLE2
Connections:
- net +15V: now also IC5.4 (V+)
- net -15V: now also IC5.11 (V-)
- net A renamed ECVA
- net ECVA: no longer J3.2 (T)
- new net ECVB: J3.2 (T)
Other:
- moved on the sheet: C3, C4

Commit message: rev a for vc-lfos module
Parts:
- J2: Legend ECVA -> ECV1
- J3: Legend ECVB -> ECV2
Changed lines of the file:
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@@
 			)
 		)
-		(property "Legend" "ECVB"
+		(property "Legend" "ECV2"
 			(at 220.98 41.2749 0)
 			(show_name no)
@@
 			)
 		)
-		(property "Legend" "ECVA"
+		(property "Legend" "ECV1"
 			(at 220.98 28.5749 0)
 			(show_name no)
