File: modules/ENVELOPE_FOLLOWER/ENVELOPE_FOLLOWER.kicad_sch (KiCad schematic)
At the start: 30 parts, among them IC1 TL074, P1 10k, P2 10k, P3 1k

Commit message: added missing gate & env selectors for envelope follower
Connections:
- net ENVELOPE renamed ENV
- net TRIGGER renamed GATE
Changed lines of the file:
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@@
 		)
 	)
-	(global_label "TRIGGER"
+	(global_label "GATE"
 		(shape output)
 		(at 130.81 139.7 0)
@@
 		)
 		(property "Intersheetrefs" "${INTERSHEET_REFS}"
-			(at 141.6917 139.7 0)
+			(at 138.3655 139.7 0)
 			(hide yes)
 			(show_name no)
@@
 		)
 	)
-	(global_label "ENVELOPE"
+	(global_label "ENV"
 		(shape output)
 		(at 231.14 78.74 0)
@@
 		)
 		(property "Intersheetrefs" "${INTERSHEET_REFS}"
-			(at 243.715 78.74 0)
+			(at 237.7884 78.74 0)
 			(hide yes)
 			(show_name no)
