File: system/BACKPLANE_A/BACKPLANE_A.kicad_sch (KiCad schematic)
At the start: 6 parts, among them J1 SLOT 1A, J2 SLOT 2A, J3 SLOT 3A, J4 SLOT 4A, J5 SLOT 5A, J6 SLOT 6A

Commit message: buss a refinements
Other:
- title: BACKPLANE A -> BACKPLANE-A
Changed lines of the file:
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@@
 	(paper "USLetter")
 	(title_block
-		(title "BACKPLANE A")
-		(date "2026-06-09")
+		(title "BACKPLANE-A")
+		(date "2026-07-20")
 		(rev "A")
 		(company "THE HOUSE OF GALAHAD")
-		(comment 1 "FORMANT-KO")
+		(comment 1 "FORMANT^{KO}")
 	)
 	(global_label "ENV3"
