File: modules/COM/system.kicad_sch (KiCad schematic)
At the start: 17 parts, among them J1 Card_Connector, J3 GATE LED, J4 IS INPUT, J5 Mono_Jack, J6 Mono_Jack, U1 RC4136

Commit message: com rework; channel first stab at schematic
Parts:
- removed D4: Panel_LED, FormantKO:Panel_Connector_1x02, symbol FormantKO:Panel_LED
- removed J3: GATE LED, FormantKO:Jumper_1x03, symbol FormantKO:Jumper_01x03
- removed J4: IS INPUT, FormantKO:Jumper_1x03, symbol FormantKO:Jumper_01x03
- removed R23: 150R, FormantKO:R_Axial_Horizontal, symbol FormantKO:R
- added D4: GATE1 LED, FormantKO:PanelConnector_1x02, symbol FormantKO:D_LED
- added D5: GATE2 LED, FormantKO:PanelConnector_1x02, symbol FormantKO:D_LED
- added J2: IS SELECT, Connector_PinHeader_2.54mm:PinHeader_2x08_P2.54mm_Vertical, symbol Connector_Generic:Conn_02x08_Odd_Even
- added R24, R27: 150R, FormantKO:R_Axial_Horizontal, symbol FormantKO:R
- added R25, R26: 10k, FormantKO:R_Axial_Horizontal, symbol FormantKO:R
- added T1, T2: 2N3904, FormantKO:TO-92, symbol Transistor_BJT:2N3904
- C11, C12: footprint FormantKO:C_Disc -> FormantKO:C_Rect_300_400
- D1: value Panel_LED -> -15V LED; footprint FormantKO:Panel_Connector_1x02 -> FormantKO:PanelConnector_1x02; symbol FormantKO:Panel_LED -> FormantKO:D_LED
- D2: value Panel_LED -> +5V LED; footprint FormantKO:Panel_Connector_1x02 -> FormantKO:PanelConnector_1x02; symbol FormantKO:Panel_LED -> FormantKO:D_LED
- D3: value Panel_LED -> +15V LED; footprint FormantKO:Panel_Connector_1x02 -> FormantKO:PanelConnector_1x02; symbol FormantKO:Panel_LED -> FormantKO:D_LED
- J1: value Card_Connector -> CardConnector; footprint FormantKO:Card_Connector -> FormantKO:CardConnector; symbol FormantKO:Card_Connector -> FormantKO:CardConnector
- J5: value Mono_Jack -> OUT 1; footprint FormantKO:Panel_Connector_1x02 -> FormantKO:PanelConnector_1x02; symbol FormantKO:Mono_Jack -> FormantKO:MonoJack
- J6: value Mono_Jack -> OUT 2; footprint FormantKO:Panel_Connector_1x02 -> FormantKO:PanelConnector_1x02; symbol FormantKO:Mono_Jack -> FormantKO:MonoJack
- MH1: footprint FormantKO:Card_Bracket -> FormantKO:CardBracket; symbol FormantKO:Card_Bracket -> FormantKO:CardBracket
Connections:
- net +5V: now also R24.2, R27.2
- net GATE1: now also R25.1
- net GATE2: now also R26.1
- net GND: now also T1.1 (E), T2.1 (E)
- net IS: now also J2.1 (Pin_1), J2.11 (Pin_11), J2.13 (Pin_13), J2.15 (Pin_15), J2.3 (Pin_3), J2.5 (Pin_5), J2.7 (Pin_7), J2.9 (Pin_9)
- net VCA1: now also J2.14 (Pin_14)
- net VCA2: now also J2.16 (Pin_16)
- net VCO1: now reaches J1.a24 (VCO1)
- net VCO1: now also J2.2 (Pin_2)
- net VCO3: now reaches J1.a26 (VCO3)
- net VCO3: now also J2.6 (Pin_6)
- net VCF1: now reaches J1.a28 (VCF1)
- net VCF1: now also J2.10 (Pin_10)
- net VCO2: now reaches J1.b24 (VCO2)
- net VCO2: now also J2.4 (Pin_4)
- net RFM: now reaches J1.b26 (RFM)
- net RFM: now also J2.8 (Pin_8)
- net VCF2: now reaches J1.b28 (VCF2)
- net VCF2: now also J2.12 (Pin_12)
- new net: R26.2, T2.2 (B)
- new net: R25.2, T1.2 (B)
- new net: D4.1 (K), T1.3 (C)
- new net: D5.1 (K), T2.3 (C)
- new net: D5.2 (A), R27.1
- new net: D4.2 (A), R24.1
- no-connect marks 12 -> 6
Other:
- moved on the sheet: J1, J6, MH1

Commit message: com pcb update
Connections:
- net +15V: now also C11.2; no longer C11.1
- net -15V: now also C12.1; no longer C12.2
- net GND: now also C11.1, C12.2; no longer C11.2, C12.1
Other:
- moved on the sheet: C11, C12
Changed lines of the file:
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@@
 	)
 	(junction
+		(at 63.5 96.52)
+		(diameter 0)
+		(color 0 0 0 0)
+	)
+	(junction
 		(at 45.72 140.97)
 		(diameter 0)
@@
 	)
 	(junction
-		(at 63.5 96.52)
-		(diameter 0)
-		(color 0 0 0 0)
-	)
-	(junction
 		(at 45.72 137.16)
 		(diameter 0)
@@
 	(symbol
 		(lib_id "FormantKO:C")
-		(at 63.5 92.71 0)
+		(at 63.5 92.71 180)
 		(unit 1)
 		(body_style 1)
@@
 					(size 1.27 1.27)
 				)
-				(justify left)
+				(justify right)
 			)
 		)
@@
 					(size 1.27 1.27)
 				)
-				(justify left)
+				(justify right)
 			)
 		)
@@
 	(symbol
 		(lib_id "FormantKO:C")
-		(at 63.5 100.33 0)
+		(at 63.5 100.33 180)
 		(unit 1)
 		(body_style 1)
@@
 					(size 1.27 1.27)
 				)
-				(justify left)
+				(justify right)
 			)
 		)
@@
 					(size 1.27 1.27)
 				)
-				(justify left)
+				(justify right)
 			)
 		)

Commit message: com updates for new templates and styles
Parts:
- added J10: P2.3, FormantKO:Wire_1x01_General, symbol FormantKO:Wire_1x01
- added J11: OUT 2, FormantKO:Wire_1x01_General, symbol FormantKO:Wire_1x01
- added J12: P3.1, FormantKO:Wire_1x01_General, symbol FormantKO:Wire_1x01
- added J13: P3.2, FormantKO:Wire_1x01_General, symbol FormantKO:Wire_1x01
- added J14: P3.3, FormantKO:Wire_1x01_General, symbol FormantKO:Wire_1x01
- added J15, J20, J22, J28, J32: GND, FormantKO:Wire_1x01_General, symbol FormantKO:Wire_1x01
- added J16: P1b.1, FormantKO:Wire_1x01_General, symbol FormantKO:Wire_1x01
- added J17: P1b.2, FormantKO:Wire_1x01_General, symbol FormantKO:Wire_1x01
- added J18: P1b.3, FormantKO:Wire_1x01_General, symbol FormantKO:Wire_1x01
- added J19: OUT 1, FormantKO:Wire_1x01_General, symbol FormantKO:Wire_1x01
- added J21: -15V, FormantKO:Wire_1x01_General, symbol FormantKO:Wire_1x01
- added J23: 5V LED, FormantKO:Wire_1x01_General, symbol FormantKO:Wire_1x01
- added J24: +15V LED, FormantKO:Wire_1x01_General, symbol FormantKO:Wire_1x01
- added J25: -15V LED, FormantKO:Wire_1x01_General, symbol FormantKO:Wire_1x01
- added J26: GATE1 LED, FormantKO:Wire_1x01_General, symbol FormantKO:Wire_1x01
- added J27: GATE2 LED, FormantKO:Wire_1x01_General, symbol FormantKO:Wire_1x01
- added J29: P4.1, FormantKO:Wire_1x01_General, symbol FormantKO:Wire_1x01
- added J3: P1a.1, FormantKO:Wire_1x01_General, symbol FormantKO:Wire_1x01
- added J30: P4.2, FormantKO:Wire_1x01_General, symbol FormantKO:Wire_1x01
- added J31: P4.3, FormantKO:Wire_1x01_General, symbol FormantKO:Wire_1x01
- added J4: P1a.2, FormantKO:Wire_1x01_General, symbol FormantKO:Wire_1x01
- added J7: P1a.3, FormantKO:Wire_1x01_General, symbol FormantKO:Wire_1x01
- added J8: P2.1, FormantKO:Wire_1x01_General, symbol FormantKO:Wire_1x01
- added J9: P2.2, FormantKO:Wire_1x01_General, symbol FormantKO:Wire_1x01
- renumbered U1 to IC1
Connections:
- net -15V: now also J21.1 (Pin_1)
- net GND: now also J15.1 (Pin_1), J20.1 (Pin_1), J22.1 (Pin_1), J28.1 (Pin_1), J32.1 (Pin_1)
- net IOS: now also J19.1 (Pin_1)
- net PA: now also J11.1 (Pin_1)
- net -15V LED: now reaches D1.2 (A), R20.2
- net -15V LED: now also J25.1 (Pin_1)
- net GATE2 LED: now reaches D5.2 (A), R27.1
- net GATE2 LED: now also J27.1 (Pin_1)
- net +15V LED: now reaches D3.2 (A), R22.2
- net +15V LED: now also J24.1 (Pin_1)
- net GATE1 LED: now reaches D4.2 (A), R24.1
- net GATE1 LED: now also J26.1 (Pin_1)
- net 5V LED: now reaches D2.2 (A), R21.2
- net 5V LED: now also J23.1 (Pin_1)
- new net P1A.1: J3.1 (Pin_1)
- new net P1A.2: J4.1 (Pin_1)
- new net P1A.3: J7.1 (Pin_1)
- new net P1B.1: J16.1 (Pin_1)
- new net P1B.2: J17.1 (Pin_1)
- new net P1B.3: J18.1 (Pin_1)
- new net P2.1: J8.1 (Pin_1)
- new net P2.2: J9.1 (Pin_1)
- new net P2.3: J10.1 (Pin_1)
- new net P3.1: J12.1 (Pin_1)
- new net P3.2: J13.1 (Pin_1)
- new net P3.3: J14.1 (Pin_1)
- new net P4.1: J29.1 (Pin_1)
- new net P4.2: J30.1 (Pin_1)
- new net P4.3: J31.1 (Pin_1)
Other:
- note added: "WIRE PADS"
- moved on the sheet: D1, D2, D3, D4, D5, J5, J6, R20, R21, R22, R24, R25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
