File: modules/TEMPLATE/system.kicad_sch (KiCad schematic)
At the start: 2 parts, among them J1 Card_Connector

Commit message: com revamp
Parts:
- J1: value Card_Connector -> Card Connector
- MH1: value CardBracket -> Card Bracket
Other:
- note added: "BUS AND I/O CONFIGURATION"
- note added: "PANEL HARDWARE"
- note added: "POWER DECOUPLING"
- note added: "WIRE PADS"
- moved on the sheet: J1, MH1
