File: modules/POWER_SUPPLIES/BIPOLAR_PSU/BIPOLAR_PSU.kicad_pcb (KiCad board)
At the start: 2 copper layers, 106 x 32 mm, 22 parts, among them IC1 L7815, IC2 L7915, J1 AC1, J2 AC2, J3 +, J4 0, J5 -, J6 ACG

Commit message: bipolar project cleanup
Parts:
- D1, D2, D3, D4: value 1N4001 -> type="" model="1N4001" lib="semiconductor.lib"
- J1: value AC1 -> AC
- J2: value AC2 -> AC
- J6: value ACG -> CT
Routing:
- added copper zone on F.Cu, net GND
Other:
- board text added: "| ${COMMENT2} | ${COMMENT3} |"
- board text removed: "${COMMENT2} ${COMMENT3}"
