File: MFOS/modules/CALIBRATOR/system.kicad_sch (KiCad schematic)
At the start: 7 parts, among them J1 Card Connector, U1 40106, U2 4520

Commit message: calibrator pcb done
Parts:
- added C2, C8: 10μ, FormantKO:CP_Radial_P100mil, symbol FormantKO:C_Polarized
- added C3, C4, C6, C7: 100n, FormantKO:C_Rect_P200mil, symbol FormantKO:C
- added X10, X8, X9: WireConnector, FormantKO:Wire_1x01_D40mil_OD80mil, symbol FormantKO:WireConnector
- C1: footprint FormantKO:CP_Axial_P600mil -> FormantKO:CP_Radial_P100mil; Voltage 16V -> 25V
- J2: renamed from J1; footprint FormantKO:Card_Connector -> FormantKO:CardConnector; symbol FormantKO:Card_Connector -> FormantKO:CardConnector
- MH1: footprint FormantKO:Card_Bracket -> FormantKO:CardBracket; symbol FormantKO:Card_Bracket -> FormantKO:CardBracket
- Z1: Spice_Lib_File semiconductor.lib -> (none); Spice_Node_Sequence 2 1 -> (none)
Connections:
- net +15V: now also C2.1, C3.1, C4.1, X8.1
- net -15V: now also C6.2, C7.2, C8.2, X10.1
- net GND: now also C2.2, C3.2, C4.2, C6.1, C7.1, C8.1, X9.1
Other:
- note added: "9V POWER"
- title: TEMPLATE -> MFOS CALIBRATOR
- moved on the sheet: C1, R2, Z1
