File: MFOS/modules/EXPANDER/EXPANDER.kicad_pcb (KiCad board)
At the start: 2 copper layers, 160 x 100 mm, 37 parts, among them IC1 TL074, IC2 TL074, IC3 TL074, J1 Card Connector, J2 MonoJack, J3 MonoJack, J4 MonoJack, J5 MonoJack, J6 MonoJack, J7 MonoJack, J8 MonoJack, U1 40106, X12 WireConnector, X2 WireConnector, X22 WireConnector, X3 WireConnector, X4 WireConnector, X7 WireConnector

Commit message: work on mfos expander
Parts:
- removed J2, J3, J4, J5, J6, J7, J8: MonoJack, FormantKO:PanelConnector_1x02
- removed S1: SW, FormantKO:PanelConnector_1x03
- removed U1: 40106, FormantKO:DIP-14N
- added C1: 10µ, FormantKO:CP_Radial_P100mil, F.Cu at (197.2, 84.8)
- added C2: 220n, FormantKO:C_Rect_P200mil, F.Cu at (175.6, 59.4)
- added C3: 10µ, FormantKO:CP_Radial_P100mil, F.Cu at (198.5, 109.0)
- added C4: 1µ, FormantKO:CP_Radial_P100mil, F.Cu at (198.5, 98.8)
- added C7: 47p, FormantKO:C_Rect_P200mil, F.Cu at (122.3, 96.3)
- added C8: 220n, FormantKO:C_Rect_P200mil, F.Cu at (141.3, 116.6)
- added D1: 1N4148, FormantKO:DO-35_P400mil, F.Cu at (165.5, 121.7)
- added D2: 1N4148, FormantKO:DO-35_P400mil, F.Cu at (128.7, 112.8)
- added D3: 1N4148, FormantKO:DO-35_P400mil, F.Cu at (117.2, 116.6)
- added IC4: 40106, FormantKO:DIP-14N, F.Cu at (161.7, 107.7)
- added J12: KOV SELECT, Connector_PinHeader_2.54mm:PinHeader_2x02_P2.54mm_Vertical, F.Cu at (194.7, 55.6)
- added J14: GATE SELECT, Connector_PinHeader_2.54mm:PinHeader_2x02_P2.54mm_Vertical, F.Cu at (194.7, 64.5)
- added R11: 10k, FormantKO:R_Axial_Horizontal_P500mil, F.Cu at (185.8, 74.7)
- added R12: 100k, FormantKO:R_Axial_Horizontal_P500mil, F.Cu at (149.0, 121.7)
- added R13: 100R, FormantKO:R_Axial_Horizontal_P500mil, F.Cu at (154.1, 116.6)
- added R15: 1k, FormantKO:R_Axial_Horizontal_P500mil, F.Cu at (145.2, 105.0)
- added R16: 10k, FormantKO:R_Axial_Horizontal_P500mil, F.Cu at (180.7, 74.7)
- added R17: 20k, FormantKO:R_Axial_Horizontal_P500mil, F.Cu at (138.8, 101.3)
- added R18: 130k, FormantKO:R_Axial_Horizontal_P500mil, F.Cu at (149.0, 125.5)
- added R19: 2k, FormantKO:R_Axial_Horizontal_P500mil, F.Cu at (175.6, 120.4)
- added R20: 1M, FormantKO:R_Axial_Horizontal_P500mil, F.Cu at (117.2, 100.1)
- added R21: 100k, FormantKO:R_Axial_Horizontal_P500mil, F.Cu at (180.7, 120.4)
- added R22: 100k, FormantKO:Potentiometer_Trimmer_MultiTurn, F.Cu at (133.7, 125.5)
- added R23: 10k, FormantKO:R_Axial_Horizontal_P500mil, F.Cu at (103.2, 121.7)
- added R24: 100k, FormantKO:R_Axial_Horizontal_P500mil, F.Cu at (127.4, 116.6)
- added R25: 10k, FormantKO:R_Axial_Horizontal_P500mil, F.Cu at (103.2, 126.8)
- added R26: 2k, FormantKO:R_Axial_Horizontal_P500mil, F.Cu at (175.6, 102.6)
- added R27: 20k, FormantKO:R_Axial_Horizontal_P500mil, F.Cu at (133.7, 101.3)
- added R28: 130k, FormantKO:R_Axial_Horizontal_P500mil, F.Cu at (128.7, 101.3)
- added R29: 10k, FormantKO:R_Axial_Horizontal_P500mil, F.Cu at (103.2, 131.8)
- added R7: 100R, FormantKO:R_Axial_Horizontal_P500mil, F.Cu at (160.4, 59.4)
- added R9: 10k, FormantKO:R_Axial_Horizontal_P500mil, F.Cu at (151.5, 78.5)
- added T1: 2N3904, FormantKO:TO-92_Wide, F.Cu at (188.3, 124.2)
- added X1: WireConnector, FormantKO:Wire_1x01_D40mil_OD80mil, F.Cu at (67.7, 69.6)
- added X10: WireConnector, FormantKO:Wire_1x01_D40mil_OD80mil, F.Cu at (75.3, 92.5)
- added X11: WireConnector, FormantKO:Wire_1x01_D40mil_OD80mil, F.Cu at (67.7, 95.0)
- added X13: WireConnector, FormantKO:Wire_1x01_D40mil_OD80mil, F.Cu at (67.7, 100.1)
- added X14: WireConnector, FormantKO:Wire_1x01_D40mil_OD80mil, F.Cu at (75.3, 102.6)
- added X15: WireConnector, FormantKO:Wire_1x01_D40mil_OD80mil, F.Cu at (67.7, 105.2)
- added X16: WireConnector, FormantKO:Wire_1x01_D40mil_OD80mil, F.Cu at (75.3, 107.7)
- added X17: WireConnector, FormantKO:Wire_1x01_D40mil_OD80mil, F.Cu at (67.7, 110.2)
- added X18: WireConnector, FormantKO:Wire_1x01_D40mil_OD80mil, F.Cu at (75.3, 112.8)
- added X19: WireConnector, FormantKO:Wire_1x01_D40mil_OD80mil, F.Cu at (67.7, 115.3)
- added X20: WireConnector, FormantKO:Wire_1x01_D40mil_OD80mil, F.Cu at (75.3, 117.9)
- added X21: WireConnector, FormantKO:Wire_1x01_D40mil_OD80mil, F.Cu at (67.7, 120.4)
- added X5: WireConnector, FormantKO:Wire_1x01_D40mil_OD80mil, F.Cu at (67.7, 79.8)
- added X6: WireConnector, FormantKO:Wire_1x01_D40mil_OD80mil, F.Cu at (75.3, 82.3)
- added X8: WireConnector, FormantKO:Wire_1x01_D40mil_OD80mil, F.Cu at (75.3, 87.4)
- added X9: WireConnector, FormantKO:Wire_1x01_D40mil_OD80mil, F.Cu at (67.7, 89.9)
- Z2, Z4: value 1N5231 -> type="" model="1N5231" lib="semiconductor.lib"
- moved X3 95.4 mm to (67.7, 74.7)
- moved X22 72.2 mm to (75.3, 122.9)
- moved X12 51.7 mm to (75.3, 97.5)
- moved X7 41.7 mm to (67.7, 84.8)
- moved X4 39.7 mm to (75.3, 77.2)
- moved Z2 22.9 mm to (91.8, 65.8), turned to 0 degrees
- moved X2 15.3 mm to (75.3, 72.1)
- moved C10 13.3 mm to (165.5, 92.5)
- moved Z4 9.92 mm to (105.8, 65.8), turned to 180 degrees
- moved R1 9.92 mm to (86.7, 78.5)
- moved R8 9.16 mm to (91.8, 78.5), turned to -90 degrees
- moved Z3 9.16 mm to (140.1, 65.8)
- moved R3 9.16 mm to (140.1, 59.4)
- moved IC1 8.52 mm to (121.0, 78.5)
- moved R10 8.52 mm to (96.9, 78.5), turned to -90 degrees
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Connections:
- net CVBUF renamed PORTCV
- C11 pad 1: -15V -> +15V
- C5 pad 1: -15V -> +15V
- C9 pad 1: -15V -> +15V
- IC2 pad 1: unconnected-(IC2-Pad1) -> Net-(IC2A--)
- IC2 pad 12: unconnected-(IC2D-+-Pad12) -> Net-(IC2D-+)
- IC2 pad 13: unconnected-(IC2D---Pad13) -> Net-(IC2D--)
- IC2 pad 14: unconnected-(IC2-Pad14) -> Net-(IC2D--)
- IC2 pad 2: unconnected-(IC2A---Pad2) -> Net-(IC2A--)
- IC2 pad 3: unconnected-(IC2A-+-Pad3) -> Net-(IC2A-+)
- IC2 pad 5: unconnected-(IC2B-+-Pad5) -> Net-(IC2B-+)
- IC2 pad 6: unconnected-(IC2B---Pad6) -> Net-(IC2B--)
- IC2 pad 7: unconnected-(IC2-Pad7) -> Net-(IC2B--)
- IC3 pad 1: unconnected-(IC3-Pad1) -> Net-(D3-A)
- IC3 pad 10: unconnected-(IC3C-+-Pad10) -> Net-(IC3C-+)
- IC3 pad 12: unconnected-(IC3D-+-Pad12) -> Net-(IC3D-+)
- IC3 pad 13: unconnected-(IC3D---Pad13) -> Net-(IC3D--)
- IC3 pad 14: unconnected-(IC3-Pad14) -> Net-(IC3D--)
- IC3 pad 2: unconnected-(IC3A---Pad2) -> Net-(IC3A--)
- IC3 pad 3: unconnected-(IC3A-+-Pad3) -> Net-(IC3A-+)
- IC3 pad 5: unconnected-(IC3B-+-Pad5) -> Net-(IC3B-+)
- IC3 pad 6: unconnected-(IC3B---Pad6) -> Net-(IC3B--)
- IC3 pad 7: unconnected-(IC3-Pad7) -> Net-(IC3B--)
- IC3 pad 8: unconnected-(IC3-Pad8) -> Net-(IC3C--)
- IC3 pad 9: unconnected-(IC3C---Pad9) -> Net-(IC3C--)
- J1 pad a2: unconnected-(J1-KOV1-Pada2) -> KOV1
- J1 pad a4: unconnected-(J1-GATE1-Pada4) -> GATE1
- J1 pad b2: unconnected-(J1-KOV2-Padb2) -> KOV2
- J1 pad b4: unconnected-(J1-GATE2-Padb4) -> GATE2
Routing:
- net Net-(IC1A--): track 0.00 -> 57.2 mm
- net Net-(IC1B-+): track 0.00 -> 36.8 mm
- net CV-1: track 0.00 -> 36.8 mm
- net Net-(IC1A-+): track 0.00 -> 36.8 mm
- net GND: track 0.00 -> 34.3 mm
- net Net-(IC1D-+): track 0.00 -> 29.2 mm
- net Net-(Z2-K-): track 0.00 -> 26.7 mm
- net Net-(R22-Pad2): track 0.00 -> 10.2 mm
- net Net-(R1-Pad1): track 0.00 -> 5.08 mm
- net Net-(Z2-A+): track 0.00 -> 3.81 mm
Other:
- board text added: "GATE1"
- board text added: "GATE2"
- board text added: "KOV1"
- board text added: "KOV2"
