File: panels/TEMPLATE_6U/TEMPLATE_6U.kicad_pcb (KiCad board)
At the start: 2 copper layers, 70.8 x 261.8 mm, 6 parts

Commit message: work on mfos expander
Other:
- board text added: "${COMMENT1}"
- board text added: "${COMPANY} ${COMMENT4}"
- board text added: "${TITLE} ${COMMENT5} REVISION ${REVISION} ${CURRENT_DATE}"
- board text removed: "${COMPANY} ${TAG}"
- board text removed: "${MODULE} ${PARTNO} REVISION ${REVISION} ${ISSUE_DATE}"
- board text removed: "FORMANT^{KO}"
Changed lines of the file:
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@@
 	(title_block
 		(title "TEMPLATE 6U")
-		(date "2026-06-05")
+		(date "9999-99-99")
 		(rev "A")
 		(company "THE HOUSE OF GALAHAD")
 		(comment 1 "FORMANT^{KO}")
+		(comment 2 "mailto:paul.f.burdette@gmail.com")
+		(comment 3 "https://github.com/Desval27/FormantKO/")
+		(comment 4 "No Organic Grounding")
+		(comment 5 "0000-Z")
 	)
 	(layers
@@
 		)
 	)
-	(gr_text "FORMANT^{KO}"
+	(gr_text "${COMMENT1}"
 		(at 201.635894 276.115428 0)
 		(layer "F.SilkS")
@@
 		)
 	)
-	(gr_text "${MODULE} ${PARTNO}\nREVISION ${REVISION} ${ISSUE_DATE}"
+	(gr_text "${TITLE} ${COMMENT5}\nREVISION ${REVISION} ${CURRENT_DATE}"
 		(at 201.635894 276.115428 0)
 		(layer "B.SilkS")
@@
 		)
 	)
-	(gr_text "${COMPANY}\n${TAG}"
+	(gr_text "${COMPANY}\n${COMMENT4}"
 		(at 201.645894 24.365428 0)
 		(layer "B.SilkS")
